Commit message: Add README, refine xacro.

File: grizzly_ur10_description/urdf/base_with_manipulator.urdf.xacro (robot description, xacro)
@@ -26,14 +26,5 @@
 -->
 <robot xmlns:xacro="http://ros.org/wiki/xacro" name="grizzly_ur10">
-  <xacro:property name="reflect" value="-1" />
   <xacro:include filename="$(find grizzly_description)/urdf/base.urdf.xacro" />
-  <xacro:include filename="$(find ur_description)/urdf/gazebo.urdf.xacro" />
-  <xacro:include filename="$(find ur_description)/urdf/ur10.urdf.xacro" />
-  <!-- Spawn arm -->
-  <xacro:ur10_robot prefix="arm_" joint_limited="true" />
-  <joint name="grizzly_ur10_joint" type="fixed">
-    <parent link="sensor_anchor_link" />
-    <child link="arm_base_link" />
-    <origin xyz="0.65 ${reflect * 0.21} 0.03" rpy="0.0 0.0 ${-pi/2}" />
-  </joint>
+  <xacro:include filename="$(find grizzly_ur10_description)/urdf/manipulator.urdf.xacro" />
 </robot>
