Commit message: Update physical and collision properties

File: grizzly_description/urdf/add_frame.urdf.xacro (robot description, xacro)
@@ -29,34 +29,6 @@
 -->
 <robot name="grizzly_tf" xmlns:xacro="http://www.ros.org/wiki/xacro">
-  <property name="x_com"
-            value="0.00000000" />
-  <!-- com : center of mass -->
-  <property name="y_com"
-            value="0.00000000" />
-  <!-- com : center of mass -->
-  <property name="z_com"
-            value="0.00000000" />
-  <!-- com : center of mass -->
-  <property name="mass"
-            value="0.1" />
-  <!-- in kg-->
-  <property name="ixx_com_cs"
-            value="0.01" />
-  <!-- at center of mass aligned with coordinate system, kg*m^2-->
-  <property name="ixy_com_cs"
-            value="0.0" />
-  <!-- at center of mass aligned with coordinate system, kg*m^2-->
-  <property name="ixz_com_cs"
-            value="0.0" />
-  <!-- at center of mass aligned with coordinate system, kg*m^2-->
-  <property name="iyy_com_cs"
-            value="0.01" />
-  <!-- at center of mass aligned with coordinate system, kg*m^2-->
-  <property name="iyz_com_cs"
-            value="0.00" />
-  <!-- at center of mass aligned with coordinate system, kg*m^2-->
-  <property name="izz_com_cs"
-            value="0.01" />
-  <!-- at center of mass aligned with coordinate system, kg*m^2-->
+  <property name="mass" value="0.01" />
+  <property name="dummy_inertia" value="1e-09"/>
   <xacro:macro name="grizzly_tf"
                params="parent name translateX translateY translateZ rotateX rotateY rotateZ">
@@ -71,11 +43,11 @@
       <inertial>
         <mass value="${mass}" />
-        <origin xyz="${x_com} ${y_com} ${z_com}" />
-        <inertia ixx="${ixx_com_cs}"
-                 ixy="${ixy_com_cs}"
-                 ixz="${ixz_com_cs}"
-                 iyy="${iyy_com_cs}"
-                 iyz="${iyz_com_cs}"
-                 izz="${izz_com_cs}" />
+        <origin xyz="0 0 0" />
+        <inertia ixx="${dummy_inertia}"
+                 ixy="0.0"
+                 ixz="0.0"
+                 iyy="${dummy_inertia}"
+                 iyz="0.0"
+                 izz="${dummy_inertia}" />
       </inertial>
     </link>

File: grizzly_description/urdf/base.urdf.xacro (robot description, xacro)
@@ -41,21 +41,18 @@
             value="-0.013" />
   <property name="base_y_com"
-            value="-0.061" />
+            value="-0.00061" />
   <property name="base_z_com"
             value="-0.0205" />
-  <!-- Size of the base-->
-  <property name="base_x_size"
-            value="0.708" />
-  <property name="base_y_size"
-            value="0.3" />
-  <property name="base_z_size"
-            value="1.826" />
+  <property name="chassis_length" value="1.75" />
+  <property name="chassis_width" value="0.711" />
+  <property name="chassis_height" value="0.495" />
   <!-- Mass of the base-->
   <property name="base_mass" value="487" />
   <!-- Mass of the front axle-->
   <property name="front_axle_mass" value="113" />
-  <!--Inertial values for the front_axle at center of mass, aligned with coordinate system. Units are kg*m^2-->
-  <!-- Ix = Iz = m*(3r^2 + h^2)/12 -->
-  <!-- Iy = m*r^2/2 -->
+  <property name="front_axle_radius" value="0.13" />
+  <property name="front_axle_length" value="1.0" />
+  <!-- Moments of inertia. Taken at center of mass aligned with coordinate system, kg*m^2-->
+  <!-- Ix = Iz = m*(3r^2 + h^2)/12   Iy = m*r^2/2-->
   <property name="front_axle_ixx_com_cs"
             value="9.9" />
@@ -65,10 +62,9 @@
             value="0.0" />
   <property name="front_axle_iyy_com_cs"
-            value="0.95" />
+            value="9.9" />
   <property name="front_axle_iyz_com_cs"
             value="0.0" />
   <property name="front_axle_izz_com_cs"
-            value="9.9" />
-  <!--Inertial values for the base at center of mass, aligned with coordinate system. Units are kg*m^2-->
+            value="0.95" />
   <property name="base_ixx_com_cs"
             value="64.010712692" />
@@ -83,23 +79,20 @@
   <property name="base_izz_com_cs"
             value="229.831441333" />
-  <!-- BASE-FOOTPRINT -->
-  <!-- base_footprint is a fictitious link(frame) that is on the ground right below base_link origin, navigation stack depends on this frame -->
-  <link name="base_footprint" />
-  <joint name="base_footprint_joint"
+  <!-- BASE-LINK -->
+  <link name="base_link" />
+  <joint name="base_link_joint"
          type="fixed">
-    <origin xyz="0 0 ${wheel_x_size/2}"
-            rpy="0 0 0"/>
-    <parent link="base_footprint" />
-    <child link="base_link" />
+    <origin xyz="0 0 0"
+            rpy="0 0 ${ground_clearance}"/>
+    <parent link="base_link" />
+    <child link="chassis_link" />
   </joint>
-  <!-- BASE-LINK -->
+  <!-- CHASSIS-LINK -->
   <!--Actual body/chassis of the robot-->
-  <link name="base_link">
+  <link name="chassis_link">
     <inertial>
       <mass value="${base_mass}" />
-      <!--This is the pose of the inertial reference frame, relative to the link reference frame. The origin of the inertial reference frame needs to be at the center of gravity. The axes of the inertial reference frame do not need to be aligned with the principal axes of the inertia.-->
       <!-- Center of mass -->
       <origin xyz="${base_x_com} ${base_y_com} ${base_z_com}" />
-      <!--The 3x3 rotational inertia matrix. Because the rotational inertia matrix is symmetric, only 6 above-diagonal elements of this matrix are specified here, using the attributes ixx, ixy, ixz, iyy, iyz, izz.-->
       <inertia ixx="${base_ixx_com_cs}"
                ixy="${base_ixy_com_cs}"
@@ -110,5 +103,5 @@
     </inertial>
     <visual>
-      <origin xyz="0 0 ${base_z_origin_offset}"
+      <origin xyz="0 0 ${ground_clearance}"
               rpy="${M_PI/2} 0 ${M_PI/2}" />
       <geometry>
@@ -118,9 +111,8 @@
     </visual>
     <collision>
-      <origin xyz="0 0 0.3"
+      <origin xyz="0 0 ${ground_clearance}"
               rpy="${M_PI/2} 0 ${M_PI/2}" />
       <geometry>
-        <box size="${base_x_size} ${base_y_size} ${base_z_size}" />
-        <!--making it slightly bigger in x and z direction-->
+         <box size="${chassis_width} ${chassis_height} ${chassis_length}"/>
       </geometry>
     </collision>
@@ -128,30 +120,33 @@
   <!-- Add a sensor anchor link that points to the center of the robot top plate -->
   <grizzly_tf parent="base_link" name="sensor_anchor_link"
-    translateX="0" translateY="0" translateZ="0.45"
-    rotateX="0.0" rotateY="0.0" rotateZ="0.0"/>
+    translateX="0" translateY="0" translateZ="${chassis_height}"
+    rotateX="0" rotateY="0" rotateZ="0"/>
   <!-- Add a sensor anchor link for the imu -->
   <grizzly_tf parent="sensor_anchor_link" name="imu_link"
-    translateX="-0.788" translateY="0" translateZ="-0.118"
+    translateX="-${chassis_length/2}" translateY="0" translateZ="0"
     rotateX="${M_PI}" rotateY="${M_PI/2}" rotateZ="0" />
   <!-- Add a sensor anchor link for the gps -->
   <grizzly_tf parent="sensor_anchor_link" name="navsat_link"
-    translateX="-0.788" translateY="0" translateZ="-0.118"
+    translateX="-${chassis_length/2}" translateY="0" translateZ="0"
     rotateX="${M_PI}" rotateY="${M_PI/2}" rotateZ="0" />
   <!-- DECORATIONS -->
-  <!-- Bumpers -->
-  <grizzly_part parent="base_footprint"
-                name="bumper"
-                mesh="bumper"
-                colour="Yellow"
-                translateX="0.0"
-                translateY="0.0"
-                translateZ="0.5"
-                rotateX="${M_PI/2}"
-                rotateY="0.0"
-                rotateZ="${M_PI/2}" />
+  <!-- Fenders -->
+  <link name="fenders_link">
+    <visual>
+      <origin xyz="0 0 ${ground_clearance}" rpy="${M_PI/2} 0 ${M_PI/2}"/>
+      <geometry>
+        <mesh filename="package://grizzly_description/meshes/bumper.stl" />
+      </geometry>
+      <material name="Yellow" />
+    </visual>
+  </link>
+  <joint name="fenders_joint" type="fixed">
+    <parent link="chassis_link" />
+    <child link="fenders_link" />
+  </joint>
   <!-- rear wheels -->
   <grizzly_wheel fr="rear"
                  lr="left"
-                 parent="base_link"
+                 parent="chassis_link"
                  translateX="-1"
                  translateY="1"
@@ -160,5 +155,5 @@
   <grizzly_wheel fr="rear"
                  lr="right"
-                 parent="base_link"
+                 parent="chassis_link"
                  translateX="-1"
                  translateY="-1"
@@ -170,5 +165,5 @@
     <origin xyz="${base_x_origin_to_wheel_origin} 0 0"
             rpy="0 0 0" />
-    <parent link="base_link" />
+    <parent link="chassis_link" />
     <child link="front_axle_link" />
     <axis xyz="1 0 0"
@@ -191,5 +186,5 @@
     </inertial>
     <visual>
-      <origin xyz="-0.2 0 0.45"
+      <origin xyz="-${ground_clearance} 0 ${base_y_origin_to_wheel_origin}"
               rpy="0 ${M_PI} ${M_PI/2}" />
       <geometry>
@@ -202,6 +197,6 @@
               rpy="${M_PI/2} 0 0" />
       <geometry>
-        <cylinder length="1.0"
-                  radius="0.13" />
+        <cylinder length="${front_axle_length}"
+                  radius="${front_axle_radius}" />
       </geometry>
     </collision>

File: grizzly_description/urdf/parts.urdf.xacro (robot description, xacro)
@@ -29,40 +29,26 @@
 -->
 <robot name="grizzly_part" xmlns:xacro="http://www.ros.org/wiki/xacro">
-  <property name="x_com"
-            value="0.00000000" />
-  <!-- com : center of mass -->
-  <property name="y_com"
-            value="0.00000000" />
-  <!-- com : center of mass -->
-  <property name="z_com"
-            value="0.00000000" />
-  <!-- com : center of mass -->
   <property name="x_size"
-            value="1.0" />
+            value="0.01" />
   <property name="y_size"
-            value="1.0" />
+            value="0.01" />
   <property name="z_size"
-            value="1.0" />
+            value="0.01" />
   <property name="mass"
             value="0.1" />
   <!-- in kg-->
+  <!-- Moments of inertia. Taken at center of mass aligned with coordinate system, kg*m^2-->
   <property name="ixx_com_cs"
             value="0.01" />
-  <!-- at center of mass aligned with coordinate system, kg*m^2-->
   <property name="ixy_com_cs"
             value="0.0" />
-  <!-- at center of mass aligned with coordinate system, kg*m^2-->
   <property name="ixz_com_cs"
             value="0.0" />
-  <!-- at center of mass aligned with coordinate system, kg*m^2-->
   <property name="iyy_com_cs"
             value="0.01" />
-  <!-- at center of mass aligned with coordinate system, kg*m^2-->
   <property name="iyz_com_cs"
             value="0.00" />
-  <!-- at center of mass aligned with coordinate system, kg*m^2-->
   <property name="izz_com_cs"
             value="0.01" />
-  <!-- at center of mass aligned with coordinate system, kg*m^2-->
   <xacro:macro name="grizzly_part"
                params="parent name mesh colour translateX translateY translateZ rotateX rotateY rotateZ">
@@ -77,6 +63,7 @@
       <inertial>
         <mass value="${mass}" />
-        <origin xyz="${x_com} ${y_com} ${z_com}" />
-        <inertia ixx="${ixx_com_cs}"
+        <origin xyz="0 0 0"
+                rpy="0 0 0" />
+      <inertia ixx="${ixx_com_cs}"
                  ixy="${ixy_com_cs}"
                  ixz="${ixz_com_cs}"

File: grizzly_description/urdf/wheel.urdf.xacro (robot description, xacro)
@@ -29,47 +29,37 @@
             value="3.14159" />
   <!-- Wheel -->
+  <property name="wheel_mass" value="15" />
+  <property name="wheel_radius"
+            value="0.33" />
+  <property name="wheel_width"
+            value="0.252" />
+  <!-- com : center of mass -->
   <property name="wheel_x_com"
             value="-0.002" />
-  <!-- com : center of mass -->
   <property name="wheel_y_com"
             value="-0.198" />
-  <!-- com : center of mass -->
   <property name="wheel_z_com"
             value="0.003" />
-  <!-- com : center of mass -->
-  <property name="wheel_x_size"
-            value="0.66" />
-  <property name="wheel_y_size"
-            value="0.66" />
-  <property name="wheel_z_size"
-            value="0.252" />
-  <property name="wheel_mass" value="15" />
+  <!-- Moments of inertia. Taken at center of mass aligned with coordinate system, kg*m^2-->
   <property name="wheel_ixx_com_cs"
             value="14.68" />
-  <!-- at center of mass aligned with coordinate system, kg*m^2-->
   <property name="wheel_ixy_com_cs"
             value="-0.033" />
-  <!-- at center of mass aligned with coordinate system, kg*m^2-->
   <property name="wheel_ixz_com_cs"
             value="0.070" />
-  <!-- at center of mass aligned with coordinate system, kg*m^2-->
   <property name="wheel_iyy_com_cs"
             value="26.7" />
-  <!-- at center of mass aligned with coordinate system, kg*m^2-->
   <property name="wheel_iyz_com_cs"
             value="-0.05" />
-  <!-- at center of mass aligned with coordinate system, kg*m^2-->
   <property name="wheel_izz_com_cs"
             value="14.68" />
-  <!-- at center of mass aligned with coordinate system, kg*m^2-->
   <property name="base_x_origin_to_wheel_origin"
-            value="0.448" />
+            value="0.448" /> <!-- 240/2 + 660/2-->
   <property name="base_y_origin_to_wheel_origin"
-            value="0.499" />
+            value="0.499" /> <!--(1282-711)/4 + 711/2-->
   <property name="base_z_origin_to_wheel_origin"
             value="0.0" />
-  <property name="base_z_origin_offset"
-            value="0.2" />
-  <!-- origin is offset in + z direction by 3.175mm, so need to bring it back down for visual and collision-->
+  <property name="ground_clearance"
+            value="0.203" />
   <xacro:macro name="grizzly_wheel"
                params="fr lr parent translateX translateY translateZ flipY">
@@ -98,12 +88,12 @@
                 rpy="${M_PI/2} ${flipY*M_PI} 0" />
         <geometry>
-          <cylinder length="${wheel_z_size}"
-                    radius="${wheel_x_size/2}" />
+          <cylinder length="${wheel_width}"
+                    radius="${wheel_radius}" />
         </geometry>
       </collision>
     </link>
     <gazebo reference="${fr}_${lr}_wheel">
-      <mu1 value="100.0" />
-      <mu2 value="0.1" />
+      <mu1 value="1.0" />
+      <mu2 value="1.0" />
       <kp value="10000000.0" />
       <kd value="1.0" />
@@ -129,8 +119,9 @@
     <transmission name="joint_${fr}_${lr}_wheel_trans"
                   type="SimpleTransmission">
-      <actuator name="joint_${fr}_${lr}_wheel_motor" />
+      <actuator name="joint_${fr}_${lr}_wheel_motor" >
+          <mechanicalReduction>1</mechanicalReduction>
+          <motorTorqueConstant>1</motorTorqueConstant>
+      </actuator>
       <joint name="joint_${fr}_${lr}_wheel" />
-      <mechanicalReduction>1</mechanicalReduction>
-      <motorTorqueConstant>1</motorTorqueConstant>
     </transmission>
   </xacro:macro>
