Commit message: move the Media/models to the meshes/ folder to keep consistent with other gazebo repos, added front axel simulation, and rewired URDF frames such that the colors show up right in Gazebo

File: grizzly_description/urdf/base.urdf.xacro (robot description, xacro)
@@ -26,22 +26,22 @@
 -->
 <robot
-	xmlns:xi="http://www.w3.org/2001/XInclude"
-	xmlns:gazebo="http://playerstage.sourceforge.net/gazebo/xmlschema/#gz"
+    xmlns:xi="http://www.w3.org/2001/XInclude"
+    xmlns:gazebo="http://playerstage.sourceforge.net/gazebo/xmlschema/#gz"
     xmlns:model="http://playerstage.sourceforge.net/gazebo/xmlschema/#model"
-	xmlns:sensor="http://playerstage.sourceforge.net/gazebo/xmlschema/#sensor"
-	xmlns:body="http://playerstage.sourceforge.net/gazebo/xmlschema/#body"
+    xmlns:sensor="http://playerstage.sourceforge.net/gazebo/xmlschema/#sensor"
+    xmlns:body="http://playerstage.sourceforge.net/gazebo/xmlschema/#body"
     xmlns:geom="http://playerstage.sourceforge.net/gazebo/xmlschema/#geom"
     xmlns:joint="http://playerstage.sourceforge.net/gazebo/xmlschema/#joint"
-	xmlns:controller="http://playerstage.sourceforge.net/gazebo/xmlschema/#controller"
-	xmlns:interface="http://playerstage.sourceforge.net/gazebo/xmlschema/#interface"
-	xmlns:rendering="http://playerstage.sourceforge.net/gazebo/xmlschema/#rendering"
+    xmlns:controller="http://playerstage.sourceforge.net/gazebo/xmlschema/#controller"
+    xmlns:interface="http://playerstage.sourceforge.net/gazebo/xmlschema/#interface"
+    xmlns:rendering="http://playerstage.sourceforge.net/gazebo/xmlschema/#rendering"
     xmlns:renderable="http://playerstage.sourceforge.net/gazebo/xmlschema/#renderable"
     xmlns:physics="http://playerstage.sourceforge.net/gazebo/xmlschema/#physics"
-	xmlns:xacro="http://ros.org/wiki/xacro" name="grizzly">
-	<!-- Included URDF/XACRO Files -->
-    <include filename="$(find grizzly_description)/urdf/materials.urdf.xacro" />
-    <include filename="$(find grizzly_description)/urdf/wheel.urdf.xacro" />
-    <include filename="$(find grizzly_description)/urdf/parts.urdf.xacro" />
-	<!-- PROPERTY LIST -->
+    xmlns:xacro="http://ros.org/wiki/xacro" name="grizzly">
+    <!-- Included URDF/XACRO Files -->
+    <xacro:include filename="$(find grizzly_description)/urdf/materials.urdf.xacro" />
+    <xacro:include filename="$(find grizzly_description)/urdf/wheel.urdf.xacro" />
+    <xacro:include filename="$(find grizzly_description)/urdf/parts.urdf.xacro" />
+    <!-- PROPERTY LIST -->
     <!--All units in m-kg-s-radians unit system -->
     <property name="M_PI" value="3.1415926535897931" />
@@ -53,8 +53,17 @@
     <!-- Size of the base-->
     <property name="base_x_size" value="0.708" />
-    <property name="base_y_size" value="0.656" />
+    <property name="base_y_size" value="0.3" />
     <property name="base_z_size" value="1.826"/>
     <!--Weight of the base-->
     <property name="base_mass" value="33.45489000" /> <!-- in kg-->
+    <!--Weight of the front axel-->
+    <property name="front_axel_mass" value="0.45489000" /> <!-- in kg-->
+    <!--Inertial values for the front_axel at center of mass, aligned with coordinate system. Units are kg*m^2-->
+    <property name="front_axel_ixx_com_cs" value="0.60216370" />
+    <property name="front_axel_ixy_com_cs" value="-0.02364198" />
+    <property name="front_axel_ixz_com_cs" value="-0.11972132" />
+    <property name="front_axel_iyy_com_cs" value="1.73859574" />
+    <property name="front_axel_iyz_com_cs" value="-0.00154437" />
+    <property name="front_axel_izz_com_cs" value="2.02955229" />
     <!--Inertial values for the base at center of mass, aligned with coordinate system. Units are kg*m^2-->
     <property name="base_ixx_com_cs" value="0.60216370" />
@@ -82,5 +91,4 @@
     </link>
     <gazebo reference="base_footprint">
-        <material>Gazebo/Green</material>
         <turnGravityOff>false</turnGravityOff>
     </gazebo>
@@ -104,14 +112,14 @@
             <origin xyz="0 0 ${base_z_origin_offset}" rpy="${M_PI/2} 0 ${M_PI/2}" />
             <geometry>
-                <mesh filename="package://grizzly_description/Media/models/base_link.stl" />
+                <mesh filename="package://grizzly_description/meshes/base_link.stl" />
             </geometry>
             <material name="Black" />
         </visual>
-		<collision>
-			<origin xyz="0 0 ${base_z_origin_offset}" rpy="${M_PI/2} 0 ${M_PI/2}" />
-			<geometry>
-				<box size = "${base_x_size} ${base_y_size} ${base_z_size + 0.02}"/> <!--making it slightly bigger in x and z direction-->
-			</geometry>
-		</collision>
+        <collision>
+            <origin xyz="0 0 0.3" rpy="${M_PI/2} 0 ${M_PI/2}" />
+            <geometry>
+                <box size = "${base_x_size} ${base_y_size} ${base_z_size}"/> <!--making it slightly bigger in x and z direction-->
+            </geometry>
+        </collision>
     </link>
     <gazebo reference="base_link">
@@ -119,30 +127,66 @@
         <turnGravityOff>false</turnGravityOff>
     </gazebo>
-    <!-- WHEEL macros -->
-	<grizzly_wheel fb="back" lr="left" parent="base_link" translateX="-1.75" translateY="1.75" flipY="0"/>
-	<grizzly_wheel fb="back" lr="right" parent="base_link" translateX="-1.75" translateY="-1.75" flipY="1"/>
-	<grizzly_wheel fb="front" lr="left" parent="base_link" translateX="1.75" translateY="1.75" flipY="0"/>
-	<grizzly_wheel fb="front" lr="right" parent="base_link" translateX="1.75" translateY="-1.75" flipY="1"/>
     <!-- DECORATIONS -->
     <!-- Bumpers -->
-    <grizzly_part parent="base_link" name="bumper" mesh="bumper"
+    <grizzly_part parent="base_footprint" name="bumper" mesh="bumper"
           colour="Yellow"
-          translateX="0.0" translateY="0.0" translateZ="${base_z_origin_offset}"
+          translateX="0.0" translateY="0.0" translateZ="0.5"
           rotateX="${M_PI/2}" rotateY="0.0" rotateZ="${M_PI/2}"/>
-    <gazebo reference="base_link_bumper_part">
+    <gazebo reference="base_footprint_bumper_part">
         <material>Gazebo/Yellow</material>
     </gazebo>
+    <!-- Back wheels -->
+	<grizzly_wheel fb="back" lr="left" parent="base_link" translateX="-1.75" translateY="1.75" translateZ="0" flipY="0"/>
+	<grizzly_wheel fb="back" lr="right" parent="base_link" translateX="-1.75" translateY="-1.75" translateZ="0" flipY="1"/>
+    <!-- Front wheels -->
+    <joint name="front_axel_joint" type="revolute">
+		<origin xyz="0.4375 0 0" rpy="0 0 0" />
+        <parent link="base_link"/>
+        <child link="front_axel_link" />
+        <axis xyz="1 0 0" rpy="0 0 0" />
+        <limit effort="10" lower="-0.2" upper="0.2" velocity="0.5"/>
+    </joint>
+    <!-- Front axel link -->
+    <link name="front_axel_link">
+        <inertial>
+            <mass value="${front_axel_mass}" />
+            <origin xyz="0 0 0" />
+            <inertia ixx="${front_axel_ixx_com_cs}" ixy="${front_axel_ixy_com_cs}" ixz="${front_axel_ixz_com_cs}"
+                iyy="${front_axel_iyy_com_cs}" iyz="${front_axel_iyz_com_cs}" izz="${front_axel_izz_com_cs}" />
+        </inertial>
+        <visual>
+            <origin xyz="0 0 0" rpy="${M_PI/2} 0 0" />
+            <geometry>
+                <!--mesh filename="package://grizzly_description/meshes/front_axel_link.stl" /-->
+				<cylinder length="1.0" radius="0.13" />
+            </geometry>
+            <material name="Black" />
+        </visual>
+        <collision>
+            <origin xyz="0 0 0" rpy="${M_PI/2} 0 0" />
+            <geometry>
+				<cylinder length="1.0" radius="0.13" />
+            </geometry>
+        </collision>
+    </link>
+    <gazebo reference="front_axel_link">
+        <material>Gazebo/FlatBlack</material>
+        <turnGravityOff>false</turnGravityOff>
+    </gazebo>
+	<grizzly_wheel fb="front" lr="left" parent="front_axel_link" translateX="0" translateY="1.75" translateZ="0" flipY="0"/>
+	<grizzly_wheel fb="front" lr="right" parent="front_axel_link" translateX="0" translateY="-1.75" translateZ="0" flipY="1"/>
     <gazebo>
-		<controller:grizzly_plugin name="grizzly_diff_controller" plugin="libgrizzly_gazebo_plugins.so">
-		        <alwaysOn>true</alwaysOn>
-		        <updateRate>100.0</updateRate>
-		        <backLeftJoint>joint_back_left_wheel</backLeftJoint>
-		        <backRightJoint>joint_back_right_wheel</backRightJoint>
-		        <frontLeftJoint>joint_front_left_wheel</frontLeftJoint>
-		        <frontRightJoint>joint_front_right_wheel</frontRightJoint>
-		        <wheelSeparation>${base_y_size}</wheelSeparation>
-		        <wheelDiameter>${wheel_x_size}</wheelDiameter>
-		        <torque>35</torque>
-        </controller:grizzly_plugin>
-	</gazebo>
+	    <plugin name="grizzly_diff_controller" filename="libgrizzly_gazebo_plugins.so">
+            <alwaysOn>true</alwaysOn>
+            <updateRate>100.0</updateRate>
+            <backLeftJoint>joint_back_left_wheel</backLeftJoint>
+            <backRightJoint>joint_back_right_wheel</backRightJoint>
+            <frontLeftJoint>joint_front_left_wheel</frontLeftJoint>
+            <frontRightJoint>joint_front_right_wheel</frontRightJoint>
+            <frontAxelJoint>front_axel_joint</frontAxelJoint>
+            <wheelSeparation>${base_y_size}</wheelSeparation>
+            <wheelDiameter>${wheel_x_size}</wheelDiameter>
+            <torque>35</torque>
+        </plugin>
+    </gazebo>
 </robot>

File: grizzly_description/urdf/parts.urdf.xacro (robot description, xacro)
@@ -62,5 +62,5 @@
 				<origin xyz="0 0 0" rpy="0 0 0" />
 				<geometry>
-					<mesh filename="package://grizzly_description/Media/models/${mesh}.stl" />
+					<mesh filename="package://grizzly_description/meshes/${mesh}.stl" />
 				</geometry>
 				<material name="${colour}" />

File: grizzly_description/urdf/wheel.urdf.xacro (robot description, xacro)
@@ -29,72 +29,72 @@
 	xmlns:interface="http://playerstage.sourceforge.net/gazebo/xmlschema/#interface"
 	xmlns:xacro="http://ros.org/wiki/xacro" name="grizzly_wheel">
-	<property name="M_PI" value="3.14159"/>
-	<!-- Wheel -->
-	<property name="wheel_x_com" value="0.00000000" /> <!-- com : center of mass -->
-	<property name="wheel_y_com" value="0.00000000" /> <!-- com : center of mass -->
-	<property name="wheel_z_com" value="0.00019000" /> <!-- com : center of mass -->
-	<property name="wheel_x_size" value="0.66" />
-	<property name="wheel_y_size" value="0.66" />
-	<property name="wheel_z_size" value="0.252" />
-	<property name="wheel_mass" value="2.63657000" /> <!-- in kg-->
-	<property name="wheel_ixx_com_cs" value="0.02466885" /> <!-- at center of mass aligned with coordinate system, kg*m^2-->
-	<property name="wheel_ixy_com_cs" value="0.00000000" /> <!-- at center of mass aligned with coordinate system, kg*m^2-->
-	<property name="wheel_ixz_com_cs" value="0.00000000" /> <!-- at center of mass aligned with coordinate system, kg*m^2-->
-	<property name="wheel_iyy_com_cs" value="0.02466885" /> <!-- at center of mass aligned with coordinate system, kg*m^2-->
-	<property name="wheel_iyz_com_cs" value="0.00000000" /> <!-- at center of mass aligned with coordinate system, kg*m^2-->
-	<property name="wheel_izz_com_cs" value="0.04410576" /> <!-- at center of mass aligned with coordinate system, kg*m^2-->
-	<property name="base_x_origin_to_wheel_origin" value="0.25600006" />
-	<property name="base_y_origin_to_wheel_origin" value="0.285475" />
-	<property name="base_z_origin_to_wheel_origin" value="0.0" />
-	<property name="base_z_origin_offset" value="0.2" /> <!-- origin is offset in + z direction by 3.175mm, so need to bring it back down for visual and collision-->
-	<xacro:macro name="grizzly_wheel" params="fb lr parent translateX translateY flipY"> <!--fb : front, back ; lr: left, right -->
-		<link name="${fb}_${lr}_wheel">
-			<inertial>
-				<mass value="${wheel_mass}" />
-				<origin xyz="${wheel_x_com} ${wheel_y_com} ${wheel_z_com}" />
-				<inertia  ixx="${wheel_ixx_com_cs}" ixy="${wheel_ixy_com_cs}" ixz="${wheel_ixz_com_cs}"
-					iyy="${wheel_iyy_com_cs}" iyz="${wheel_iyz_com_cs}" izz="${wheel_izz_com_cs}" />
-			</inertial>
-			<visual>
-				<origin xyz="0 0 0" rpy="${M_PI/2} ${flipY*M_PI} ${M_PI/2}" />
-				<geometry>
-					<mesh filename="package://grizzly_description/Media/models/wheel.stl" />
-				</geometry>
-				<material name="DarkGray" />
-			</visual>
-			<collision>
-				<origin xyz="0 0 0" rpy="${M_PI/2} ${flipY*M_PI} 0" />
-				<geometry>
-				    <cylinder length="${wheel_z_size}" radius="${wheel_x_size/2}" />
-				<!--
-					<mesh filename="package://husky_description/Media/models/wheel.stl" />
-			    -->
-				</geometry>
-			</collision>
-		</link>
-		<gazebo reference="${fb}_${lr}_wheel">
-			<mu1 value="1.0"/>
-			<mu2 value="1.0"/>
-			<kp  value="100000.0" />
-			<kd  value="1.0" />
-			<fdir1 value="1 0 0"/>
-			<material>Gazebo/Grey</material>
-			<turnGravityOff>false</turnGravityOff>
-		</gazebo>
-		<joint name="joint_${fb}_${lr}_wheel" type="continuous">
-			<parent link="${parent}"/>
-			<child link="${fb}_${lr}_wheel"/>
-			<origin xyz="${translateX * base_x_origin_to_wheel_origin} ${translateY * base_y_origin_to_wheel_origin} ${base_z_origin_to_wheel_origin}" rpy="0 0 0" />
-			<axis xyz="0 1 0" rpy="0 0 0" />
-			<limit effort="100" velocity="100"/>
-			<joint_properties damping="0.0" friction="0.0"/>
-		</joint>
-		<!-- Transmission is important to link the joints and the controller -->
-		<transmission name="joint_${fb}_${lr}_wheel_trans" type="SimpleTransmission">
-			<actuator name="joint_${fb}_${lr}_wheel_motor" />
-			<joint name="joint_${fb}_${lr}_wheel" />
-			<mechanicalReduction>1</mechanicalReduction>
-			<motorTorqueConstant>1</motorTorqueConstant>
-		</transmission>
+    <property name="M_PI" value="3.14159"/>
+    <!-- Wheel -->
+    <property name="wheel_x_com" value="0.00000000" /> <!-- com : center of mass -->
+    <property name="wheel_y_com" value="0.00000000" /> <!-- com : center of mass -->
+    <property name="wheel_z_com" value="0.00019000" /> <!-- com : center of mass -->
+    <property name="wheel_x_size" value="0.66" />
+    <property name="wheel_y_size" value="0.66" />
+    <property name="wheel_z_size" value="0.252" />
+    <property name="wheel_mass" value="2.63657000" /> <!-- in kg-->
+    <property name="wheel_ixx_com_cs" value="0.02466885" /> <!-- at center of mass aligned with coordinate system, kg*m^2-->
+    <property name="wheel_ixy_com_cs" value="0.00000000" /> <!-- at center of mass aligned with coordinate system, kg*m^2-->
+    <property name="wheel_ixz_com_cs" value="0.00000000" /> <!-- at center of mass aligned with coordinate system, kg*m^2-->
+    <property name="wheel_iyy_com_cs" value="0.02466885" /> <!-- at center of mass aligned with coordinate system, kg*m^2-->
+    <property name="wheel_iyz_com_cs" value="0.00000000" /> <!-- at center of mass aligned with coordinate system, kg*m^2-->
+    <property name="wheel_izz_com_cs" value="0.04410576" /> <!-- at center of mass aligned with coordinate system, kg*m^2-->
+    <property name="base_x_origin_to_wheel_origin" value="0.25600006" />
+    <property name="base_y_origin_to_wheel_origin" value="0.285475" />
+    <property name="base_z_origin_to_wheel_origin" value="0.0" />
+    <property name="base_z_origin_offset" value="0.2" /> <!-- origin is offset in + z direction by 3.175mm, so need to bring it back down for visual and collision-->
+	<xacro:macro name="grizzly_wheel" params="fb lr parent translateX translateY translateZ flipY"> <!--fb : front, back ; lr: left, right -->
+        <link name="${fb}_${lr}_wheel">
+            <inertial>
+                <mass value="${wheel_mass}" />
+                <origin xyz="${wheel_x_com} ${wheel_y_com} ${wheel_z_com}" />
+                <inertia  ixx="${wheel_ixx_com_cs}" ixy="${wheel_ixy_com_cs}" ixz="${wheel_ixz_com_cs}"
+                    iyy="${wheel_iyy_com_cs}" iyz="${wheel_iyz_com_cs}" izz="${wheel_izz_com_cs}" />
+            </inertial>
+            <visual>
+                <origin xyz="0 0 0" rpy="${M_PI/2} ${flipY*M_PI} ${M_PI/2}" />
+                <geometry>
+                    <mesh filename="package://grizzly_description/meshes/wheel.stl" />
+                </geometry>
+                <material name="DarkGray" />
+            </visual>
+            <collision>
+                <origin xyz="0 0 0" rpy="${M_PI/2} ${flipY*M_PI} 0" />
+                <geometry>
+                    <cylinder length="${wheel_z_size}" radius="${wheel_x_size/2}" />
+                <!--
+                    <mesh filename="package://husky_description/Media/models/wheel.stl" />
+                -->
+                </geometry>
+            </collision>
+        </link>
+        <gazebo reference="${fb}_${lr}_wheel">
+            <mu1 value="100.0"/>
+            <mu2 value="0.1"/>
+            <kp  value="10000000.0" />
+            <kd  value="1.0" />
+            <fdir1 value="1 0 0"/>
+            <material>Gazebo/Grey</material>
+            <turnGravityOff>false</turnGravityOff>
+        </gazebo>
+        <joint name="joint_${fb}_${lr}_wheel" type="continuous">
+            <parent link="${parent}"/>
+            <child link="${fb}_${lr}_wheel"/>
+            <origin xyz="${translateX * base_x_origin_to_wheel_origin} ${translateY * base_y_origin_to_wheel_origin} ${translateZ}" rpy="0 0 0" />
+            <axis xyz="0 1 0" rpy="0 0 0" />
+            <limit effort="100" velocity="100"/>
+            <joint_properties damping="0.0" friction="0.0"/>
+        </joint>
+        <!-- Transmission is important to link the joints and the controller -->
+        <transmission name="joint_${fb}_${lr}_wheel_trans" type="SimpleTransmission">
+            <actuator name="joint_${fb}_${lr}_wheel_motor" />
+            <joint name="joint_${fb}_${lr}_wheel" />
+            <mechanicalReduction>1</mechanicalReduction>
+            <motorTorqueConstant>1</motorTorqueConstant>
+        </transmission>
   	</xacro:macro>
 </robot>

Commit message: adding new downsampled meshes, and changed the front axel joint parameters to make the visualization work

File: grizzly_description/urdf/base.urdf.xacro (robot description, xacro)
@@ -156,8 +156,7 @@
         </inertial>
         <visual>
-            <origin xyz="0 0 0" rpy="${M_PI/2} 0 0" />
+            <origin xyz="-0.2 0 0.45" rpy="0 ${M_PI} ${M_PI/2}" />
             <geometry>
-                <!--mesh filename="package://grizzly_description/meshes/front_axel_link.stl" /-->
-				<cylinder length="1.0" radius="0.13" />
+                <mesh filename="package://grizzly_description/meshes/front_axel.stl" />
             </geometry>
             <material name="Black" />
