Commit message: Fix tabbing and formatting.

File: grizzly_description/urdf/base.urdf.xacro (robot description, xacro)
@@ -25,167 +25,247 @@
 This program contains the description of the robot base model for the Clearpath Grizzly
 -->
-<robot
-    xmlns:xi="http://www.w3.org/2001/XInclude"
-    xmlns:gazebo="http://playerstage.sourceforge.net/gazebo/xmlschema/#gz"
-    xmlns:model="http://playerstage.sourceforge.net/gazebo/xmlschema/#model"
-    xmlns:sensor="http://playerstage.sourceforge.net/gazebo/xmlschema/#sensor"
-    xmlns:body="http://playerstage.sourceforge.net/gazebo/xmlschema/#body"
-    xmlns:geom="http://playerstage.sourceforge.net/gazebo/xmlschema/#geom"
-    xmlns:joint="http://playerstage.sourceforge.net/gazebo/xmlschema/#joint"
-    xmlns:controller="http://playerstage.sourceforge.net/gazebo/xmlschema/#controller"
-    xmlns:interface="http://playerstage.sourceforge.net/gazebo/xmlschema/#interface"
-    xmlns:rendering="http://playerstage.sourceforge.net/gazebo/xmlschema/#rendering"
-    xmlns:renderable="http://playerstage.sourceforge.net/gazebo/xmlschema/#renderable"
-    xmlns:physics="http://playerstage.sourceforge.net/gazebo/xmlschema/#physics"
-    xmlns:xacro="http://ros.org/wiki/xacro" name="grizzly">
-    <!-- Included URDF/XACRO Files -->
-    <xacro:include filename="$(find grizzly_description)/urdf/materials.urdf.xacro" />
-    <xacro:include filename="$(find grizzly_description)/urdf/wheel.urdf.xacro" />
-    <xacro:include filename="$(find grizzly_description)/urdf/parts.urdf.xacro" />
-    <!-- PROPERTY LIST -->
-    <!--All units in m-kg-s-radians unit system -->
-    <property name="M_PI" value="3.1415926535897931" />
-    <!-- Main Body-base-->
-    <!-- Location of com : center of mass -->
-    <property name="base_x_com" value="-0.08748000" />
-    <property name="base_y_com" value="-0.00085000" />
-    <property name="base_z_com" value="0.09947000" />
-    <!-- Size of the base-->
-    <property name="base_x_size" value="0.708" />
-    <property name="base_y_size" value="0.3" />
-    <property name="base_z_size" value="1.826"/>
-    <!--Weight of the base-->
-    <property name="base_mass" value="33.45489000" /> <!-- in kg-->
-    <!--Weight of the front axle-->
-    <property name="front_axle_mass" value="0.45489000" /> <!-- in kg-->
-    <!--Inertial values for the front_axle at center of mass, aligned with coordinate system. Units are kg*m^2-->
-    <property name="front_axle_ixx_com_cs" value="0.60216370" />
-    <property name="front_axle_ixy_com_cs" value="-0.02364198" />
-    <property name="front_axle_ixz_com_cs" value="-0.11972132" />
-    <property name="front_axle_iyy_com_cs" value="1.73859574" />
-    <property name="front_axle_iyz_com_cs" value="-0.00154437" />
-    <property name="front_axle_izz_com_cs" value="2.02955229" />
-    <!--Inertial values for the base at center of mass, aligned with coordinate system. Units are kg*m^2-->
-    <property name="base_ixx_com_cs" value="0.60216370" />
-    <property name="base_ixy_com_cs" value="-0.02364198" />
-    <property name="base_ixz_com_cs" value="-0.11972132" />
-    <property name="base_iyy_com_cs" value="1.73859574" />
-    <property name="base_iyz_com_cs" value="-0.00154437" />
-    <property name="base_izz_com_cs" value="2.02955229" />
-    <!-- BASE-FOOTPRINT -->
-    <!-- base_footprint is a fictitious link(frame) that is on the ground right below base_link origin, navigation stack depends on this frame -->
-    <link name="base_footprint">
-        <inertial>
-            <mass value="0.0001" />
-            <origin xyz="0 0 0" />
-            <inertia ixx="0.0001" ixy="0.0" ixz="0.0"
-                iyy="0.0001" iyz="0.0"
-                izz="0.0001" />
-        </inertial>
-        <visual>
-            <origin xyz="0 0 0" rpy="0 0 0" />
-            <geometry>
-                <box size="0.001 0.001 0.001" />
-            </geometry>
-        </visual>
-    </link>
-    <gazebo reference="base_footprint">
-        <turnGravityOff>false</turnGravityOff>
-    </gazebo>
-    <joint name="base_footprint_joint" type="fixed">
-		<origin xyz="0 0 ${wheel_x_size/2}" rpy="0 0 0" />
-        <parent link="base_footprint"/>
-        <child link="base_link" />
-    </joint>
-    <!-- BASE-LINK -->
-    <!--Actual body/chassis of the robot-->
-    <link name="base_link">
-        <inertial>
-            <mass value="${base_mass}" />
-            <!--This is the pose of the inertial reference frame, relative to the link reference frame. The origin of the inertial reference frame needs to be at the center of gravity. The axes of the inertial reference frame do not need to be aligned with the principal axes of the inertia.-->
-            <origin xyz="${base_x_com} ${base_y_com} ${base_z_com}" />
-            <!--The 3x3 rotational inertia matrix. Because the rotational inertia matrix is symmetric, only 6 above-diagonal elements of this matrix are specified here, using the attributes ixx, ixy, ixz, iyy, iyz, izz.-->
-            <inertia ixx="${base_ixx_com_cs}" ixy="${base_ixy_com_cs}" ixz="${base_ixz_com_cs}"
-                iyy="${base_iyy_com_cs}" iyz="${base_iyz_com_cs}" izz="${base_izz_com_cs}" />
-        </inertial>
-        <visual>
-            <origin xyz="0 0 ${base_z_origin_offset}" rpy="${M_PI/2} 0 ${M_PI/2}" />
-            <geometry>
-                <mesh filename="package://grizzly_description/meshes/base_link.stl" />
-            </geometry>
-            <material name="Black" />
-        </visual>
-        <collision>
-            <origin xyz="0 0 0.3" rpy="${M_PI/2} 0 ${M_PI/2}" />
-            <geometry>
-                <box size = "${base_x_size} ${base_y_size} ${base_z_size}"/> <!--making it slightly bigger in x and z direction-->
-            </geometry>
-        </collision>
-    </link>
-    <gazebo reference="base_link">
-        <material>Gazebo/FlatBlack</material>
-        <turnGravityOff>false</turnGravityOff>
-    </gazebo>
-    <!-- DECORATIONS -->
-    <!-- Bumpers -->
-    <grizzly_part parent="base_footprint" name="bumper" mesh="bumper"
-          colour="Yellow"
-          translateX="0.0" translateY="0.0" translateZ="0.5"
-          rotateX="${M_PI/2}" rotateY="0.0" rotateZ="${M_PI/2}"/>
-    <gazebo reference="base_footprint_bumper_part">
-        <material>Gazebo/Yellow</material>
-    </gazebo>
-    <!-- Back wheels -->
-	<grizzly_wheel fb="back" lr="left" parent="base_link" translateX="-1.75" translateY="1.75" translateZ="0" flipY="0"/>
-	<grizzly_wheel fb="back" lr="right" parent="base_link" translateX="-1.75" translateY="-1.75" translateZ="0" flipY="1"/>
-    <!-- Front wheels -->
-    <joint name="front_axle_joint" type="revolute">
-		<origin xyz="0.4375 0 0" rpy="0 0 0" />
-        <parent link="base_link"/>
-        <child link="front_axle_link" />
-        <axis xyz="1 0 0" rpy="0 0 0" />
-        <limit effort="10" lower="-0.2" upper="0.2" velocity="0.5"/>
-    </joint>
-    <!-- Front axle link -->
-    <link name="front_axle_link">
-        <inertial>
-            <mass value="${front_axle_mass}" />
-            <origin xyz="0 0 0" />
-            <inertia ixx="${front_axle_ixx_com_cs}" ixy="${front_axle_ixy_com_cs}" ixz="${front_axle_ixz_com_cs}"
-                iyy="${front_axle_iyy_com_cs}" iyz="${front_axle_iyz_com_cs}" izz="${front_axle_izz_com_cs}" />
-        </inertial>
-        <visual>
-            <origin xyz="-0.2 0 0.45" rpy="0 ${M_PI} ${M_PI/2}" />
-            <geometry>
-                <mesh filename="package://grizzly_description/meshes/front_axle.stl" />
-            </geometry>
-            <material name="Black" />
-        </visual>
-        <collision>
-            <origin xyz="0 0 0" rpy="${M_PI/2} 0 0" />
-            <geometry>
-				<cylinder length="1.0" radius="0.13" />
-            </geometry>
-        </collision>
-    </link>
-    <gazebo reference="front_axle_link">
-        <material>Gazebo/FlatBlack</material>
-        <turnGravityOff>false</turnGravityOff>
-    </gazebo>
-	<grizzly_wheel fb="front" lr="left" parent="front_axle_link" translateX="0" translateY="1.75" translateZ="0" flipY="0"/>
-	<grizzly_wheel fb="front" lr="right" parent="front_axle_link" translateX="0" translateY="-1.75" translateZ="0" flipY="1"/>
-    <gazebo>
-	    <plugin name="grizzly_diff_controller" filename="libgrizzly_gazebo_plugins.so">
-            <alwaysOn>true</alwaysOn>
-            <updateRate>100.0</updateRate>
-            <backLeftJoint>joint_back_left_wheel</backLeftJoint>
-            <backRightJoint>joint_back_right_wheel</backRightJoint>
-            <frontLeftJoint>joint_front_left_wheel</frontLeftJoint>
-            <frontRightJoint>joint_front_right_wheel</frontRightJoint>
-            <frontAxleJoint>front_axle_joint</frontAxleJoint>
-            <wheelSeparation>${base_y_size}</wheelSeparation>
-            <wheelDiameter>${wheel_x_size}</wheelDiameter>
-            <torque>35</torque>
-        </plugin>
-    </gazebo>
+<robot xmlns:xi="http://www.w3.org/2001/XInclude"
+       xmlns:gazebo="http://playerstage.sourceforge.net/gazebo/xmlschema/#gz"
+       xmlns:model="http://playerstage.sourceforge.net/gazebo/xmlschema/#model"
+       xmlns:sensor="http://playerstage.sourceforge.net/gazebo/xmlschema/#sensor"
+       xmlns:body="http://playerstage.sourceforge.net/gazebo/xmlschema/#body"
+       xmlns:geom="http://playerstage.sourceforge.net/gazebo/xmlschema/#geom"
+       xmlns:joint="http://playerstage.sourceforge.net/gazebo/xmlschema/#joint"
+       xmlns:controller="http://playerstage.sourceforge.net/gazebo/xmlschema/#controller"
+       xmlns:interface="http://playerstage.sourceforge.net/gazebo/xmlschema/#interface"
+       xmlns:rendering="http://playerstage.sourceforge.net/gazebo/xmlschema/#rendering"
+       xmlns:renderable="http://playerstage.sourceforge.net/gazebo/xmlschema/#renderable"
+       xmlns:physics="http://playerstage.sourceforge.net/gazebo/xmlschema/#physics"
+       xmlns:xacro="http://ros.org/wiki/xacro"
+       name="grizzly">
+  <!-- Included URDF/XACRO Files -->
+  <xacro:include filename="$(find grizzly_description)/urdf/materials.urdf.xacro" />
+  <xacro:include filename="$(find grizzly_description)/urdf/wheel.urdf.xacro" />
+  <xacro:include filename="$(find grizzly_description)/urdf/parts.urdf.xacro" />
+  <!-- PROPERTY LIST -->
+  <!--All units in m-kg-s-radians unit system -->
+  <property name="M_PI"
+            value="3.1415926535897931" />
+  <!-- Main Body-base-->
+  <!-- Location of com : center of mass -->
+  <property name="base_x_com"
+            value="-0.08748000" />
+  <property name="base_y_com"
+            value="-0.00085000" />
+  <property name="base_z_com"
+            value="0.09947000" />
+  <!-- Size of the base-->
+  <property name="base_x_size"
+            value="0.708" />
+  <property name="base_y_size"
+            value="0.3" />
+  <property name="base_z_size"
+            value="1.826" />
+  <!--Weight of the base-->
+  <property name="base_mass"
+            value="33.45489000" />
+  <!-- in kg-->
+  <!--Weight of the front axle-->
+  <property name="front_axle_mass"
+            value="0.45489000" />
+  <!-- in kg-->
+  <!--Inertial values for the front_axle at center of mass, aligned with coordinate system. Units are kg*m^2-->
+  <property name="front_axle_ixx_com_cs"
+            value="0.60216370" />
+  <property name="front_axle_ixy_com_cs"
+            value="-0.02364198" />
+  <property name="front_axle_ixz_com_cs"
+            value="-0.11972132" />
+  <property name="front_axle_iyy_com_cs"
+            value="1.73859574" />
+  <property name="front_axle_iyz_com_cs"
+            value="-0.00154437" />
+  <property name="front_axle_izz_com_cs"
+            value="2.02955229" />
+  <!--Inertial values for the base at center of mass, aligned with coordinate system. Units are kg*m^2-->
+  <property name="base_ixx_com_cs"
+            value="0.60216370" />
+  <property name="base_ixy_com_cs"
+            value="-0.02364198" />
+  <property name="base_ixz_com_cs"
+            value="-0.11972132" />
+  <property name="base_iyy_com_cs"
+            value="1.73859574" />
+  <property name="base_iyz_com_cs"
+            value="-0.00154437" />
+  <property name="base_izz_com_cs"
+            value="2.02955229" />
+  <!-- BASE-FOOTPRINT -->
+  <!-- base_footprint is a fictitious link(frame) that is on the ground right below base_link origin, navigation stack depends on this frame -->
+  <link name="base_footprint">
+    <inertial>
+      <mass value="0.0001" />
+      <origin xyz="0 0 0" />
+      <inertia ixx="0.0001"
+               ixy="0.0"
+               ixz="0.0"
+               iyy="0.0001"
+               iyz="0.0"
+               izz="0.0001" />
+    </inertial>
+    <visual>
+      <origin xyz="0 0 0"
+              rpy="0 0 0" />
+      <geometry>
+        <box size="0.001 0.001 0.001" />
+      </geometry>
+    </visual>
+  </link>
+  <gazebo reference="base_footprint">
+    <turnGravityOff>false</turnGravityOff>
+  </gazebo>
+  <joint name="base_footprint_joint"
+         type="fixed">
+    <origin xyz="0 0 ${wheel_x_size/2}"
+            rpy="0 0 0" />
+    <parent link="base_footprint" />
+    <child link="base_link" />
+  </joint>
+  <!-- BASE-LINK -->
+  <!--Actual body/chassis of the robot-->
+  <link name="base_link">
+    <inertial>
+      <mass value="${base_mass}" />
+      <!--This is the pose of the inertial reference frame, relative to the link reference frame. The origin of the inertial reference frame needs to be at the center of gravity. The axes of the inertial reference frame do not need to be aligned with the principal axes of the inertia.-->
+      <origin xyz="${base_x_com} ${base_y_com} ${base_z_com}" />
+      <!--The 3x3 rotational inertia matrix. Because the rotational inertia matrix is symmetric, only 6 above-diagonal elements of this matrix are specified here, using the attributes ixx, ixy, ixz, iyy, iyz, izz.-->
+      <inertia ixx="${base_ixx_com_cs}"
+               ixy="${base_ixy_com_cs}"
+               ixz="${base_ixz_com_cs}"
+               iyy="${base_iyy_com_cs}"
+               iyz="${base_iyz_com_cs}"
+               izz="${base_izz_com_cs}" />
+    </inertial>
+    <visual>
+      <origin xyz="0 0 ${base_z_origin_offset}"
+              rpy="${M_PI/2} 0 ${M_PI/2}" />
+      <geometry>
+        <mesh filename="package://grizzly_description/meshes/base_link.stl" />
+      </geometry>
+      <material name="Black" />
+    </visual>
+    <collision>
+      <origin xyz="0 0 0.3"
+              rpy="${M_PI/2} 0 ${M_PI/2}" />
+      <geometry>
+        <box size="${base_x_size} ${base_y_size} ${base_z_size}" />
+        <!--making it slightly bigger in x and z direction-->
+      </geometry>
+    </collision>
+  </link>
+  <gazebo reference="base_link">
+    <material>Gazebo/FlatBlack</material>
+    <turnGravityOff>false</turnGravityOff>
+  </gazebo>
+  <!-- DECORATIONS -->
+  <!-- Bumpers -->
+  <grizzly_part parent="base_footprint"
+                name="bumper"
+                mesh="bumper"
+                colour="Yellow"
+                translateX="0.0"
+                translateY="0.0"
+                translateZ="0.5"
+                rotateX="${M_PI/2}"
+                rotateY="0.0"
+                rotateZ="${M_PI/2}" />
+  <gazebo reference="base_footprint_bumper_part">
+    <material>Gazebo/Yellow</material>
+  </gazebo>
+  <!-- Back wheels -->
+  <grizzly_wheel fb="back"
+                 lr="left"
+                 parent="base_link"
+                 translateX="-1.75"
+                 translateY="1.75"
+                 translateZ="0"
+                 flipY="0" />
+  <grizzly_wheel fb="back"
+                 lr="right"
+                 parent="base_link"
+                 translateX="-1.75"
+                 translateY="-1.75"
+                 translateZ="0"
+                 flipY="1" />
+  <!-- Front wheels -->
+  <joint name="front_axle_joint"
+         type="revolute">
+    <origin xyz="0.4375 0 0"
+            rpy="0 0 0" />
+    <parent link="base_link" />
+    <child link="front_axle_link" />
+    <axis xyz="1 0 0"
+          rpy="0 0 0" />
+    <limit effort="10"
+           lower="-0.2"
+           upper="0.2"
+           velocity="0.5" />
+  </joint>
+  <!-- Front axle link -->
+  <link name="front_axle_link">
+    <inertial>
+      <mass value="${front_axle_mass}" />
+      <origin xyz="0 0 0" />
+      <inertia ixx="${front_axle_ixx_com_cs}"
+               ixy="${front_axle_ixy_com_cs}"
+               ixz="${front_axle_ixz_com_cs}"
+               iyy="${front_axle_iyy_com_cs}"
+               iyz="${front_axle_iyz_com_cs}"
+               izz="${front_axle_izz_com_cs}" />
+    </inertial>
+    <visual>
+      <origin xyz="-0.2 0 0.45"
+              rpy="0 ${M_PI} ${M_PI/2}" />
+      <geometry>
+        <mesh filename="package://grizzly_description/meshes/front_axle.stl" />
+      </geometry>
+      <material name="Black" />
+    </visual>
+    <collision>
+      <origin xyz="0 0 0"
+              rpy="${M_PI/2} 0 0" />
+      <geometry>
+        <cylinder length="1.0"
+                  radius="0.13" />
+      </geometry>
+    </collision>
+  </link>
+  <gazebo reference="front_axle_link">
+    <material>Gazebo/FlatBlack</material>
+    <turnGravityOff>false</turnGravityOff>
+  </gazebo>
+  <grizzly_wheel fb="front"
+                 lr="left"
+                 parent="front_axle_link"
+                 translateX="0"
+                 translateY="1.75"
+                 translateZ="0"
+                 flipY="0" />
+  <grizzly_wheel fb="front"
+                 lr="right"
+                 parent="front_axle_link"
+                 translateX="0"
+                 translateY="-1.75"
+                 translateZ="0"
+                 flipY="1" />
+  <gazebo>
+    <plugin name="grizzly_diff_controller"
+            filename="libgrizzly_gazebo_plugins.so">
+      <alwaysOn>true</alwaysOn>
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
File: grizzly_description/urdf/materials.urdf.xacro (robot description, xacro)
@@ -26,27 +26,27 @@
 -->
 <robot>
-	<material name="Black">
-		<color rgba="0.0 0.0 0.0 1.0"/>
-	</material>
-	<material name="Blue">
-		<color rgba="0.0 0.0 0.8 1.0"/>
-	</material>
-	<material name="Green">
-		<color rgba="0.0 0.8 0.0 1.0"/>
-	</material>
-	<material name="Gray">
-		<color rgba="0.7 0.7 0.7 1.0"/>
-	</material>
-	<material name="DarkGray">
-		<color rgba="0.3 0.3 0.3 1.0"/>
-	</material>
-	<material name="Red">
-		<color rgba="0.8 0.0 0.0 1.0"/>
-	</material>
-	<material name="White">
-		<color rgba="1.0 1.0 1.0 1.0"/>
-	</material>
-	<material name="Yellow">
-		<color rgba="0.8 0.8 0.0 1.0"/>
-	</material>
+  <material name="Black">
+    <color rgba="0.0 0.0 0.0 1.0" />
+  </material>
+  <material name="Blue">
+    <color rgba="0.0 0.0 0.8 1.0" />
+  </material>
+  <material name="Green">
+    <color rgba="0.0 0.8 0.0 1.0" />
+  </material>
+  <material name="Gray">
+    <color rgba="0.7 0.7 0.7 1.0" />
+  </material>
+  <material name="DarkGray">
+    <color rgba="0.3 0.3 0.3 1.0" />
+  </material>
+  <material name="Red">
+    <color rgba="0.8 0.0 0.0 1.0" />
+  </material>
+  <material name="White">
+    <color rgba="1.0 1.0 1.0 1.0" />
+  </material>
+  <material name="Yellow">
+    <color rgba="0.8 0.8 0.0 1.0" />
+  </material>
 </robot>
