Commit message: Fix tabbing and formatting.

File: grizzly_description/urdf/parts.urdf.xacro (robot description, xacro)
@@ -29,48 +29,81 @@
 -->
 <robot xmlns:sensor="http://playerstage.sourceforge.net/gazebo/xmlschema/#sensor"
-	xmlns:controller="http://playerstage.sourceforge.net/gazebo/xmlschema/#controller"
-	xmlns:interface="http://playerstage.sourceforge.net/gazebo/xmlschema/#interface"
-	xmlns:xacro="http://ros.org/wiki/xacro" name="grizzly_part">
-	<property name="x_com" value="0.00000000" /> <!-- com : center of mass -->
-	<property name="y_com" value="0.00000000" /> <!-- com : center of mass -->
-	<property name="z_com" value="0.00000000" /> <!-- com : center of mass -->
-	<property name="x_size" value="1.0" />
-	<property name="y_size" value="1.0" />
-	<property name="z_size" value="1.0" />
-	<property name="mass" value="0.1" /> <!-- in kg-->
-	<property name="ixx_com_cs" value="0.01" /> <!-- at center of mass aligned with coordinate system, kg*m^2-->
-	<property name="ixy_com_cs" value="0.0" /> <!-- at center of mass aligned with coordinate system, kg*m^2-->
-	<property name="ixz_com_cs" value="0.0" /> <!-- at center of mass aligned with coordinate system, kg*m^2-->
-	<property name="iyy_com_cs" value="0.01" /> <!-- at center of mass aligned with coordinate system, kg*m^2-->
-	<property name="iyz_com_cs" value="0.00" /> <!-- at center of mass aligned with coordinate system, kg*m^2-->
-	<property name="izz_com_cs" value="0.01" /> <!-- at center of mass aligned with coordinate system, kg*m^2-->
-	<xacro:macro name="grizzly_part" params="parent name mesh colour translateX translateY translateZ rotateX rotateY rotateZ">
-		<joint name="${parent}_${name}_joint" type="fixed">
-		    <origin xyz="${translateX} ${translateY} ${translateZ}"
-		            rpy="${rotateX} ${rotateY} ${rotateZ}" />
-		    <parent link="${parent}" />
-		    <child link="${parent}_${name}_part" />
-		</joint>
-		<link name="${parent}_${name}_part">
-			<inertial>
-				<mass value="${mass}" />
-				<origin xyz="${x_com} ${y_com} ${z_com}" />
-				<inertia ixx="${ixx_com_cs}" ixy="${ixy_com_cs}" ixz="${ixz_com_cs}"
-					iyy="${iyy_com_cs}" iyz="${iyz_com_cs}" izz="${izz_com_cs}" />
-			</inertial>
-			<visual>
-				<origin xyz="0 0 0" rpy="0 0 0" />
-				<geometry>
-					<mesh filename="package://grizzly_description/meshes/${mesh}.stl" />
-				</geometry>
-				<material name="${colour}" />
-			</visual>
-			<collision>
-				<origin xyz="0 0 0" rpy="0 0 0"/>
-				<geometry>
-					<box size="0.001 0.001 0.001" /> <!--the collision boundary for parts are taken into account by collision boundary of the base_link-->
-				</geometry>
-			</collision>
-		</link>
-  	</xacro:macro>
+       xmlns:controller="http://playerstage.sourceforge.net/gazebo/xmlschema/#controller"
+       xmlns:interface="http://playerstage.sourceforge.net/gazebo/xmlschema/#interface"
+       xmlns:xacro="http://ros.org/wiki/xacro"
+       name="grizzly_part">
+  <property name="x_com"
+            value="0.00000000" />
+  <!-- com : center of mass -->
+  <property name="y_com"
+            value="0.00000000" />
+  <!-- com : center of mass -->
+  <property name="z_com"
+            value="0.00000000" />
+  <!-- com : center of mass -->
+  <property name="x_size"
+            value="1.0" />
+  <property name="y_size"
+            value="1.0" />
+  <property name="z_size"
+            value="1.0" />
+  <property name="mass"
+            value="0.1" />
+  <!-- in kg-->
+  <property name="ixx_com_cs"
+            value="0.01" />
+  <!-- at center of mass aligned with coordinate system, kg*m^2-->
+  <property name="ixy_com_cs"
+            value="0.0" />
+  <!-- at center of mass aligned with coordinate system, kg*m^2-->
+  <property name="ixz_com_cs"
+            value="0.0" />
+  <!-- at center of mass aligned with coordinate system, kg*m^2-->
+  <property name="iyy_com_cs"
+            value="0.01" />
+  <!-- at center of mass aligned with coordinate system, kg*m^2-->
+  <property name="iyz_com_cs"
+            value="0.00" />
+  <!-- at center of mass aligned with coordinate system, kg*m^2-->
+  <property name="izz_com_cs"
+            value="0.01" />
+  <!-- at center of mass aligned with coordinate system, kg*m^2-->
+  <xacro:macro name="grizzly_part"
+               params="parent name mesh colour translateX translateY translateZ rotateX rotateY rotateZ">
+    <joint name="${parent}_${name}_joint"
+           type="fixed">
+      <origin xyz="${translateX} ${translateY} ${translateZ}"
+              rpy="${rotateX} ${rotateY} ${rotateZ}" />
+      <parent link="${parent}" />
+      <child link="${parent}_${name}_part" />
+    </joint>
+    <link name="${parent}_${name}_part">
+      <inertial>
+        <mass value="${mass}" />
+        <origin xyz="${x_com} ${y_com} ${z_com}" />
+        <inertia ixx="${ixx_com_cs}"
+                 ixy="${ixy_com_cs}"
+                 ixz="${ixz_com_cs}"
+                 iyy="${iyy_com_cs}"
+                 iyz="${iyz_com_cs}"
+                 izz="${izz_com_cs}" />
+      </inertial>
+      <visual>
+        <origin xyz="0 0 0"
+                rpy="0 0 0" />
+        <geometry>
+          <mesh filename="package://grizzly_description/meshes/${mesh}.stl" />
+        </geometry>
+        <material name="${colour}" />
+      </visual>
+      <collision>
+        <origin xyz="0 0 0"
+                rpy="0 0 0" />
+        <geometry>
+          <box size="0.001 0.001 0.001" />
+          <!--the collision boundary for parts are taken into account by collision boundary of the base_link-->
+        </geometry>
+      </collision>
+    </link>
+  </xacro:macro>
 </robot>

File: grizzly_description/urdf/sensor_tfs.urdf.xacro (robot description, xacro)
@@ -29,32 +29,59 @@
 -->
 <robot xmlns:sensor="http://playerstage.sourceforge.net/gazebo/xmlschema/#sensor"
-	xmlns:controller="http://playerstage.sourceforge.net/gazebo/xmlschema/#controller"
-	xmlns:interface="http://playerstage.sourceforge.net/gazebo/xmlschema/#interface"
-	xmlns:xacro="http://ros.org/wiki/xacro" name="grizzly_tf">
-	<property name="x_com" value="0.00000000" /> <!-- com : center of mass -->
-	<property name="y_com" value="0.00000000" /> <!-- com : center of mass -->
-	<property name="z_com" value="0.00000000" /> <!-- com : center of mass -->
-	<property name="mass" value="0.1" /> <!-- in kg-->
-	<property name="ixx_com_cs" value="0.01" /> <!-- at center of mass aligned with coordinate system, kg*m^2-->
-	<property name="ixy_com_cs" value="0.0" /> <!-- at center of mass aligned with coordinate system, kg*m^2-->
-	<property name="ixz_com_cs" value="0.0" /> <!-- at center of mass aligned with coordinate system, kg*m^2-->
-	<property name="iyy_com_cs" value="0.01" /> <!-- at center of mass aligned with coordinate system, kg*m^2-->
-	<property name="iyz_com_cs" value="0.00" /> <!-- at center of mass aligned with coordinate system, kg*m^2-->
-	<property name="izz_com_cs" value="0.01" /> <!-- at center of mass aligned with coordinate system, kg*m^2-->
-	<xacro:macro name="grizzly_tf" params="parent name translateX translateY translateZ rotateX rotateY rotateZ">
-		<joint name="${parent}_${name}_joint" type="fixed">
-		    <origin xyz="${translateX} ${translateY} ${translateZ}"
-		            rpy="${rotateX} ${rotateY} ${rotateZ}" />
-		    <parent link="${parent}" />
-		    <child link="${name}" />
-		</joint>
-		<link name="${name}">
-			<inertial>
-				<mass value="${mass}" />
-				<origin xyz="${x_com} ${y_com} ${z_com}" />
-				<inertia ixx="${ixx_com_cs}" ixy="${ixy_com_cs}" ixz="${ixz_com_cs}"
-					iyy="${iyy_com_cs}" iyz="${iyz_com_cs}" izz="${izz_com_cs}" />
-			</inertial>
-		</link>
-  	</xacro:macro>
+       xmlns:controller="http://playerstage.sourceforge.net/gazebo/xmlschema/#controller"
+       xmlns:interface="http://playerstage.sourceforge.net/gazebo/xmlschema/#interface"
+       xmlns:xacro="http://ros.org/wiki/xacro"
+       name="grizzly_tf">
+  <property name="x_com"
+            value="0.00000000" />
+  <!-- com : center of mass -->
+  <property name="y_com"
+            value="0.00000000" />
+  <!-- com : center of mass -->
+  <property name="z_com"
+            value="0.00000000" />
+  <!-- com : center of mass -->
+  <property name="mass"
+            value="0.1" />
+  <!-- in kg-->
+  <property name="ixx_com_cs"
+            value="0.01" />
+  <!-- at center of mass aligned with coordinate system, kg*m^2-->
+  <property name="ixy_com_cs"
+            value="0.0" />
+  <!-- at center of mass aligned with coordinate system, kg*m^2-->
+  <property name="ixz_com_cs"
+            value="0.0" />
+  <!-- at center of mass aligned with coordinate system, kg*m^2-->
+  <property name="iyy_com_cs"
+            value="0.01" />
+  <!-- at center of mass aligned with coordinate system, kg*m^2-->
+  <property name="iyz_com_cs"
+            value="0.00" />
+  <!-- at center of mass aligned with coordinate system, kg*m^2-->
+  <property name="izz_com_cs"
+            value="0.01" />
+  <!-- at center of mass aligned with coordinate system, kg*m^2-->
+  <xacro:macro name="grizzly_tf"
+               params="parent name translateX translateY translateZ rotateX rotateY rotateZ">
+    <joint name="${parent}_${name}_joint"
+           type="fixed">
+      <origin xyz="${translateX} ${translateY} ${translateZ}"
+              rpy="${rotateX} ${rotateY} ${rotateZ}" />
+      <parent link="${parent}" />
+      <child link="${name}" />
+    </joint>
+    <link name="${name}">
+      <inertial>
+        <mass value="${mass}" />
+        <origin xyz="${x_com} ${y_com} ${z_com}" />
+        <inertia ixx="${ixx_com_cs}"
+                 ixy="${ixy_com_cs}"
+                 ixz="${ixz_com_cs}"
+                 iyy="${iyy_com_cs}"
+                 iyz="${iyz_com_cs}"
+                 izz="${izz_com_cs}" />
+      </inertial>
+    </link>
+  </xacro:macro>
 </robot>

File: grizzly_description/urdf/wheel.urdf.xacro (robot description, xacro)
@@ -26,75 +26,120 @@
 -->
 <robot xmlns:sensor="http://playerstage.sourceforge.net/gazebo/xmlschema/#sensor"
-	xmlns:controller="http://playerstage.sourceforge.net/gazebo/xmlschema/#controller"
-	xmlns:interface="http://playerstage.sourceforge.net/gazebo/xmlschema/#interface"
-	xmlns:xacro="http://ros.org/wiki/xacro" name="grizzly_wheel">
-    <property name="M_PI" value="3.14159"/>
-    <!-- Wheel -->
-    <property name="wheel_x_com" value="0.00000000" /> <!-- com : center of mass -->
-    <property name="wheel_y_com" value="0.00000000" /> <!-- com : center of mass -->
-    <property name="wheel_z_com" value="0.00019000" /> <!-- com : center of mass -->
-    <property name="wheel_x_size" value="0.66" />
-    <property name="wheel_y_size" value="0.66" />
-    <property name="wheel_z_size" value="0.252" />
-    <property name="wheel_mass" value="2.63657000" /> <!-- in kg-->
-    <property name="wheel_ixx_com_cs" value="0.02466885" /> <!-- at center of mass aligned with coordinate system, kg*m^2-->
-    <property name="wheel_ixy_com_cs" value="0.00000000" /> <!-- at center of mass aligned with coordinate system, kg*m^2-->
-    <property name="wheel_ixz_com_cs" value="0.00000000" /> <!-- at center of mass aligned with coordinate system, kg*m^2-->
-    <property name="wheel_iyy_com_cs" value="0.02466885" /> <!-- at center of mass aligned with coordinate system, kg*m^2-->
-    <property name="wheel_iyz_com_cs" value="0.00000000" /> <!-- at center of mass aligned with coordinate system, kg*m^2-->
-    <property name="wheel_izz_com_cs" value="0.04410576" /> <!-- at center of mass aligned with coordinate system, kg*m^2-->
-    <property name="base_x_origin_to_wheel_origin" value="0.25600006" />
-    <property name="base_y_origin_to_wheel_origin" value="0.285475" />
-    <property name="base_z_origin_to_wheel_origin" value="0.0" />
-    <property name="base_z_origin_offset" value="0.2" /> <!-- origin is offset in + z direction by 3.175mm, so need to bring it back down for visual and collision-->
-	<xacro:macro name="grizzly_wheel" params="fb lr parent translateX translateY translateZ flipY"> <!--fb : front, back ; lr: left, right -->
-        <link name="${fb}_${lr}_wheel">
-            <inertial>
-                <mass value="${wheel_mass}" />
-                <origin xyz="${wheel_x_com} ${wheel_y_com} ${wheel_z_com}" />
-                <inertia  ixx="${wheel_ixx_com_cs}" ixy="${wheel_ixy_com_cs}" ixz="${wheel_ixz_com_cs}"
-                    iyy="${wheel_iyy_com_cs}" iyz="${wheel_iyz_com_cs}" izz="${wheel_izz_com_cs}" />
-            </inertial>
-            <visual>
-                <origin xyz="0 0 0" rpy="${M_PI/2} ${flipY*M_PI} ${M_PI/2}" />
-                <geometry>
-                    <mesh filename="package://grizzly_description/meshes/wheel.stl" />
-                </geometry>
-                <material name="DarkGray" />
-            </visual>
-            <collision>
-                <origin xyz="0 0 0" rpy="${M_PI/2} ${flipY*M_PI} 0" />
-                <geometry>
-                    <cylinder length="${wheel_z_size}" radius="${wheel_x_size/2}" />
-                <!--
+       xmlns:controller="http://playerstage.sourceforge.net/gazebo/xmlschema/#controller"
+       xmlns:interface="http://playerstage.sourceforge.net/gazebo/xmlschema/#interface"
+       xmlns:xacro="http://ros.org/wiki/xacro"
+       name="grizzly_wheel">
+  <property name="M_PI"
+            value="3.14159" />
+  <!-- Wheel -->
+  <property name="wheel_x_com"
+            value="0.00000000" />
+  <!-- com : center of mass -->
+  <property name="wheel_y_com"
+            value="0.00000000" />
+  <!-- com : center of mass -->
+  <property name="wheel_z_com"
+            value="0.00019000" />
+  <!-- com : center of mass -->
+  <property name="wheel_x_size"
+            value="0.66" />
+  <property name="wheel_y_size"
+            value="0.66" />
+  <property name="wheel_z_size"
+            value="0.252" />
+  <property name="wheel_mass"
+            value="2.63657000" />
+  <!-- in kg-->
+  <property name="wheel_ixx_com_cs"
+            value="0.02466885" />
+  <!-- at center of mass aligned with coordinate system, kg*m^2-->
+  <property name="wheel_ixy_com_cs"
+            value="0.00000000" />
+  <!-- at center of mass aligned with coordinate system, kg*m^2-->
+  <property name="wheel_ixz_com_cs"
+            value="0.00000000" />
+  <!-- at center of mass aligned with coordinate system, kg*m^2-->
+  <property name="wheel_iyy_com_cs"
+            value="0.02466885" />
+  <!-- at center of mass aligned with coordinate system, kg*m^2-->
+  <property name="wheel_iyz_com_cs"
+            value="0.00000000" />
+  <!-- at center of mass aligned with coordinate system, kg*m^2-->
+  <property name="wheel_izz_com_cs"
+            value="0.04410576" />
+  <!-- at center of mass aligned with coordinate system, kg*m^2-->
+  <property name="base_x_origin_to_wheel_origin"
+            value="0.25600006" />
+  <property name="base_y_origin_to_wheel_origin"
+            value="0.285475" />
+  <property name="base_z_origin_to_wheel_origin"
+            value="0.0" />
+  <property name="base_z_origin_offset"
+            value="0.2" />
+  <!-- origin is offset in + z direction by 3.175mm, so need to bring it back down for visual and collision-->
+  <xacro:macro name="grizzly_wheel"
+               params="fb lr parent translateX translateY translateZ flipY">
+    <!--fb : front, back ; lr: left, right -->
+    <link name="${fb}_${lr}_wheel">
+      <inertial>
+        <mass value="${wheel_mass}" />
+        <origin xyz="${wheel_x_com} ${wheel_y_com} ${wheel_z_com}" />
+        <inertia ixx="${wheel_ixx_com_cs}"
+                 ixy="${wheel_ixy_com_cs}"
+                 ixz="${wheel_ixz_com_cs}"
+                 iyy="${wheel_iyy_com_cs}"
+                 iyz="${wheel_iyz_com_cs}"
+                 izz="${wheel_izz_com_cs}" />
+      </inertial>
+      <visual>
+        <origin xyz="0 0 0"
+                rpy="${M_PI/2} ${flipY*M_PI} ${M_PI/2}" />
+        <geometry>
+          <mesh filename="package://grizzly_description/meshes/wheel.stl" />
+        </geometry>
+        <material name="DarkGray" />
+      </visual>
+      <collision>
+        <origin xyz="0 0 0"
+                rpy="${M_PI/2} ${flipY*M_PI} 0" />
+        <geometry>
+          <cylinder length="${wheel_z_size}"
+                    radius="${wheel_x_size/2}" />
+          <!--
                     <mesh filename="package://husky_description/Media/models/wheel.stl" />
                 -->
-                </geometry>
-            </collision>
-        </link>
-        <gazebo reference="${fb}_${lr}_wheel">
-            <mu1 value="100.0"/>
-            <mu2 value="0.1"/>
-            <kp  value="10000000.0" />
-            <kd  value="1.0" />
-            <fdir1 value="1 0 0"/>
-            <material>Gazebo/Grey</material>
-            <turnGravityOff>false</turnGravityOff>
-        </gazebo>
-        <joint name="joint_${fb}_${lr}_wheel" type="continuous">
-            <parent link="${parent}"/>
-            <child link="${fb}_${lr}_wheel"/>
-            <origin xyz="${translateX * base_x_origin_to_wheel_origin} ${translateY * base_y_origin_to_wheel_origin} ${translateZ}" rpy="0 0 0" />
-            <axis xyz="0 1 0" rpy="0 0 0" />
-            <limit effort="100" velocity="100"/>
-            <joint_properties damping="0.0" friction="0.0"/>
-        </joint>
-        <!-- Transmission is important to link the joints and the controller -->
-        <transmission name="joint_${fb}_${lr}_wheel_trans" type="SimpleTransmission">
-            <actuator name="joint_${fb}_${lr}_wheel_motor" />
-            <joint name="joint_${fb}_${lr}_wheel" />
-            <mechanicalReduction>1</mechanicalReduction>
-            <motorTorqueConstant>1</motorTorqueConstant>
-        </transmission>
-  	</xacro:macro>
+        </geometry>
+      </collision>
+    </link>
+    <gazebo reference="${fb}_${lr}_wheel">
+      <mu1 value="100.0" />
+      <mu2 value="0.1" />
+      <kp value="10000000.0" />
+      <kd value="1.0" />
+      <fdir1 value="1 0 0" />
+      <material>Gazebo/Grey</material>
+      <turnGravityOff>false</turnGravityOff>
+    </gazebo>
+    <joint name="joint_${fb}_${lr}_wheel"
+           type="continuous">
+      <parent link="${parent}" />
+      <child link="${fb}_${lr}_wheel" />
+      <origin xyz="${translateX * base_x_origin_to_wheel_origin} ${translateY * base_y_origin_to_wheel_origin} ${translateZ}"
+              rpy="0 0 0" />
+      <axis xyz="0 1 0"
+            rpy="0 0 0" />
+      <limit effort="100"
+             velocity="100" />
+      <joint_properties damping="0.0"
+                        friction="0.0" />
+    </joint>
+    <!-- Transmission is important to link the joints and the controller -->
+    <transmission name="joint_${fb}_${lr}_wheel_trans"
+                  type="SimpleTransmission">
+      <actuator name="joint_${fb}_${lr}_wheel_motor" />
+      <joint name="joint_${fb}_${lr}_wheel" />
+      <mechanicalReduction>1</mechanicalReduction>
+      <motorTorqueConstant>1</motorTorqueConstant>
+    </transmission>
+  </xacro:macro>
 </robot>

Commit message: Aesthetic fixes to grizzly URDF.

File: grizzly_description/urdf/base.urdf.xacro (robot description, xacro)
@@ -149,5 +149,5 @@
         <mesh filename="package://grizzly_description/meshes/base_link.stl" />
       </geometry>
-      <material name="Black" />
+      <material name="DarkGrey" />
     </visual>
     <collision>
@@ -161,5 +161,5 @@
   </link>
   <gazebo reference="base_link">
-    <material>Gazebo/FlatBlack</material>
+    <material>Gazebo/DarkGrey</material>
     <turnGravityOff>false</turnGravityOff>
   </gazebo>
@@ -233,5 +233,5 @@
         <mesh filename="package://grizzly_description/meshes/front_axle.stl" />
       </geometry>
-      <material name="Black" />
+      <material name="DarkGrey" />
     </visual>
     <collision>
@@ -245,5 +245,5 @@
   </link>
   <gazebo reference="front_axle_link">
-    <material>Gazebo/FlatBlack</material>
+    <material>Gazebo/DarkGrey</material>
     <turnGravityOff>false</turnGravityOff>
   </gazebo>

File: grizzly_description/urdf/wheel.urdf.xacro (robot description, xacro)
@@ -98,5 +98,5 @@
           <mesh filename="package://grizzly_description/meshes/wheel.stl" />
         </geometry>
-        <material name="DarkGray" />
+        <material name="Grey" />
       </visual>
       <collision>

Commit message: Fixes to mass, self-collide, etc.
- Update the mass values from the wrong ones copied in from Husky.
- Turn on selfCollide for better Gazebo integration with manipulators.
- Remove trivial inertia from base_footprint to avoid KDL complaints.

File: grizzly_description/urdf/base.urdf.xacro (robot description, xacro)
@@ -63,12 +63,8 @@
   <property name="base_z_size"
             value="1.826" />
-  <!--Weight of the base-->
-  <property name="base_mass"
-            value="33.45489000" />
-  <!-- in kg-->
-  <!--Weight of the front axle-->
-  <property name="front_axle_mass"
-            value="0.45489000" />
-  <!-- in kg-->
+  <!-- Mass of the base-->
+  <property name="base_mass" value="487" />
+  <!-- Mass of the front axle-->
+  <property name="front_axle_mass" value="113" />
   <!--Inertial values for the front_axle at center of mass, aligned with coordinate system. Units are kg*m^2-->
   <property name="front_axle_ixx_com_cs"
@@ -99,23 +95,5 @@
   <!-- BASE-FOOTPRINT -->
   <!-- base_footprint is a fictitious link(frame) that is on the ground right below base_link origin, navigation stack depends on this frame -->
-  <link name="base_footprint">
-    <inertial>
-      <mass value="0.0001" />
-      <origin xyz="0 0 0" />
-      <inertia ixx="0.0001"
-               ixy="0.0"
-               ixz="0.0"
-               iyy="0.0001"
-               iyz="0.0"
-               izz="0.0001" />
-    </inertial>
-    <visual>
-      <origin xyz="0 0 0"
-              rpy="0 0 0" />
-      <geometry>
-        <box size="0.001 0.001 0.001" />
-      </geometry>
-    </visual>
-  </link>
+  <link name="base_footprint" />
   <gazebo reference="base_footprint">
     <turnGravityOff>false</turnGravityOff>
@@ -163,4 +141,5 @@
     <material>Gazebo/DarkGrey</material>
     <turnGravityOff>false</turnGravityOff>
+    <selfCollide>true</selfCollide>
   </gazebo>
   <!-- Add a sensor anchor link that points to the center of the robot top plate -->

File: grizzly_description/urdf/wheel.urdf.xacro (robot description, xacro)
@@ -48,7 +48,5 @@
   <property name="wheel_z_size"
             value="0.252" />
-  <property name="wheel_mass"
-            value="2.63657000" />
-  <!-- in kg-->
+  <property name="wheel_mass" value="15" />
   <property name="wheel_ixx_com_cs"
             value="0.02466885" />
@@ -117,4 +115,5 @@
       <material>Gazebo/Grey</material>
       <turnGravityOff>false</turnGravityOff>
+      <selfCollide>true</selfCollide>
     </gazebo>
     <joint name="joint_${fb}_${lr}_wheel"
