Commit message: change joint names. use rear instead of back

File: grizzly_description/urdf/base.urdf.xacro (robot description, xacro)
@@ -166,6 +166,6 @@
     <material>Gazebo/Yellow</material>
   </gazebo>
-  <!-- Back wheels -->
-  <grizzly_wheel fb="back"
+  <!-- rear wheels -->
+  <grizzly_wheel fr="rear"
                  lr="left"
                  parent="base_link"
@@ -174,5 +174,5 @@
                  translateZ="0"
                  flipY="0" />
-  <grizzly_wheel fb="back"
+  <grizzly_wheel fr="rear"
                  lr="right"
                  parent="base_link"
@@ -228,5 +228,5 @@
   </gazebo>
   <!-- Front wheels -->
-  <grizzly_wheel fb="front"
+  <grizzly_wheel fr="front"
                  lr="left"
                  parent="front_axle_link"
@@ -235,5 +235,5 @@
                  translateZ="0"
                  flipY="0" />
-  <grizzly_wheel fb="front"
+  <grizzly_wheel fr="front"
                  lr="right"
                  parent="front_axle_link"
@@ -248,6 +248,6 @@
       <alwaysOn>true</alwaysOn>
       <updateRate>100.0</updateRate>
-      <backLeftJoint>joint_back_left_wheel</backLeftJoint>
-      <backRightJoint>joint_back_right_wheel</backRightJoint>
+      <rearLeftJoint>joint_rear_left_wheel</rearLeftJoint>
+      <rearRightJoint>joint_rear_right_wheel</rearRightJoint>
       <frontLeftJoint>joint_front_left_wheel</frontLeftJoint>
       <frontRightJoint>joint_front_right_wheel</frontRightJoint>

File: grizzly_description/urdf/wheel.urdf.xacro (robot description, xacro)
@@ -77,7 +77,7 @@
   <!-- origin is offset in + z direction by 3.175mm, so need to bring it back down for visual and collision-->
   <xacro:macro name="grizzly_wheel"
-               params="fb lr parent translateX translateY translateZ flipY">
-    <!--fb : front, back ; lr: left, right -->
-    <link name="${fb}_${lr}_wheel">
+               params="fr lr parent translateX translateY translateZ flipY">
+    <!--fr : front, rear ; lr: left, right -->
+    <link name="${fr}_${lr}_wheel">
       <inertial>
         <mass value="${wheel_mass}" />
@@ -107,5 +107,5 @@
       </collision>
     </link>
-    <gazebo reference="${fb}_${lr}_wheel">
+    <gazebo reference="${fr}_${lr}_wheel">
       <mu1 value="100.0" />
       <mu2 value="0.1" />
@@ -117,8 +117,8 @@
       <selfCollide>true</selfCollide>
     </gazebo>
-    <joint name="joint_${fb}_${lr}_wheel"
+    <joint name="joint_${fr}_${lr}_wheel"
            type="continuous">
       <parent link="${parent}" />
-      <child link="${fb}_${lr}_wheel" />
+      <child link="${fr}_${lr}_wheel" />
       <origin xyz="${translateX * base_x_origin_to_wheel_origin} ${translateY * base_y_origin_to_wheel_origin} ${translateZ}"
               rpy="0 0 0" />
@@ -131,8 +131,8 @@
     </joint>
     <!-- Transmission is important to link the joints and the controller -->
-    <transmission name="joint_${fb}_${lr}_wheel_trans"
+    <transmission name="joint_${fr}_${lr}_wheel_trans"
                   type="SimpleTransmission">
-      <actuator name="joint_${fb}_${lr}_wheel_motor" />
-      <joint name="joint_${fb}_${lr}_wheel" />
+      <actuator name="joint_${fr}_${lr}_wheel_motor" />
+      <joint name="joint_${fr}_${lr}_wheel" />
       <mechanicalReduction>1</mechanicalReduction>
       <motorTorqueConstant>1</motorTorqueConstant>

Commit message: move gazebo tags to a separate file. clear up URDF

File: grizzly_description/urdf/base.urdf.xacro (robot description, xacro)
@@ -25,23 +25,11 @@
 This program contains the description of the robot base model for the Clearpath Grizzly
 -->
-<robot xmlns:xi="http://www.w3.org/2001/XInclude"
-       xmlns:gazebo="http://playerstage.sourceforge.net/gazebo/xmlschema/#gz"
-       xmlns:model="http://playerstage.sourceforge.net/gazebo/xmlschema/#model"
-       xmlns:sensor="http://playerstage.sourceforge.net/gazebo/xmlschema/#sensor"
-       xmlns:body="http://playerstage.sourceforge.net/gazebo/xmlschema/#body"
-       xmlns:geom="http://playerstage.sourceforge.net/gazebo/xmlschema/#geom"
-       xmlns:joint="http://playerstage.sourceforge.net/gazebo/xmlschema/#joint"
-       xmlns:controller="http://playerstage.sourceforge.net/gazebo/xmlschema/#controller"
-       xmlns:interface="http://playerstage.sourceforge.net/gazebo/xmlschema/#interface"
-       xmlns:rendering="http://playerstage.sourceforge.net/gazebo/xmlschema/#rendering"
-       xmlns:renderable="http://playerstage.sourceforge.net/gazebo/xmlschema/#renderable"
-       xmlns:physics="http://playerstage.sourceforge.net/gazebo/xmlschema/#physics"
-       xmlns:xacro="http://ros.org/wiki/xacro"
-       name="grizzly">
+<robot name="grizzly" xmlns:xacro="http://www.ros.org/wiki/xacro">
   <!-- Included URDF/XACRO Files -->
-  <xacro:include filename="$(find grizzly_description)/urdf/materials.urdf.xacro" />
-  <xacro:include filename="$(find grizzly_description)/urdf/wheel.urdf.xacro" />
-  <xacro:include filename="$(find grizzly_description)/urdf/parts.urdf.xacro" />
-  <xacro:include filename="$(find grizzly_description)/urdf/add_frame.urdf.xacro" />
+  <xacro:include filename="materials.urdf.xacro" />
+  <xacro:include filename="wheel.urdf.xacro" />
+  <xacro:include filename="parts.urdf.xacro" />
+  <xacro:include filename="add_frame.urdf.xacro" />
+  <xacro:include filename="grizzly.gazebo" />
   <!-- PROPERTY LIST -->
   <!--All units in m-kg-s-radians unit system -->
@@ -96,7 +84,4 @@
   <!-- base_footprint is a fictitious link(frame) that is on the ground right below base_link origin, navigation stack depends on this frame -->
   <link name="base_footprint" />
-  <gazebo reference="base_footprint">
-    <turnGravityOff>false</turnGravityOff>
-  </gazebo>
   <joint name="base_footprint_joint"
          type="fixed">
@@ -138,9 +123,4 @@
     </collision>
   </link>
-  <gazebo reference="base_link">
-    <material>Gazebo/DarkGrey</material>
-    <turnGravityOff>false</turnGravityOff>
-    <selfCollide>false</selfCollide>
-  </gazebo>
   <!-- Add a sensor anchor link that points to the center of the robot top plate -->
   <grizzly_tf parent="base_link" name="sensor_anchor_link"
@@ -163,7 +143,4 @@
                 rotateY="0.0"
                 rotateZ="${M_PI/2}" />
-  <gazebo reference="base_footprint_bumper_part">
-    <material>Gazebo/Yellow</material>
-  </gazebo>
   <!-- rear wheels -->
   <grizzly_wheel fr="rear"
@@ -223,8 +200,4 @@
     </collision>
   </link>
-  <gazebo reference="front_axle_link">
-    <material>Gazebo/DarkGrey</material>
-    <turnGravityOff>false</turnGravityOff>
-  </gazebo>
   <!-- Front wheels -->
   <grizzly_wheel fr="front"
@@ -242,19 +215,3 @@
                  translateZ="0"
                  flipY="1" />
-  <!-- Grizzly Plugin -->
-  <gazebo>
-    <plugin name="grizzly_diff_controller"
-            filename="libgrizzly_gazebo_plugins.so">
-      <alwaysOn>true</alwaysOn>
-      <updateRate>100.0</updateRate>
-      <rearLeftJoint>joint_rear_left_wheel</rearLeftJoint>
-      <rearRightJoint>joint_rear_right_wheel</rearRightJoint>
-      <frontLeftJoint>joint_front_left_wheel</frontLeftJoint>
-      <frontRightJoint>joint_front_right_wheel</frontRightJoint>
-      <frontAxleJoint>front_axle_joint</frontAxleJoint>
-      <wheelSeparation>${base_y_size}</wheelSeparation>
-      <wheelDiameter>${wheel_x_size}</wheelDiameter>
-      <torque>35</torque>
-    </plugin>
-  </gazebo>
 </robot>

File: grizzly_description/urdf/wheel.urdf.xacro (robot description, xacro)
@@ -25,9 +25,5 @@
 This program contains the description of the robot wheel model for Clearpath Grizzly
 -->
-<robot xmlns:sensor="http://playerstage.sourceforge.net/gazebo/xmlschema/#sensor"
-       xmlns:controller="http://playerstage.sourceforge.net/gazebo/xmlschema/#controller"
-       xmlns:interface="http://playerstage.sourceforge.net/gazebo/xmlschema/#interface"
-       xmlns:xacro="http://ros.org/wiki/xacro"
-       name="grizzly_wheel">
+<robot name="grizzly_wheel" xmlns:xacro="http://ros.org/wiki/xacro">
   <property name="M_PI"
             value="3.14159" />

Commit message: update position of wheel's joints

File: grizzly_description/urdf/base.urdf.xacro (robot description, xacro)
@@ -154,6 +154,6 @@
                  lr="left"
                  parent="base_link"
-                 translateX="-1.75"
-                 translateY="1.75"
+                 translateX="-1"
+                 translateY="1"
                  translateZ="0"
                  flipY="0" />
@@ -161,6 +161,6 @@
                  lr="right"
                  parent="base_link"
-                 translateX="-1.75"
-                 translateY="-1.75"
+                 translateX="-1"
+                 translateY="-1"
                  translateZ="0"
                  flipY="1" />
@@ -168,5 +168,5 @@
   <joint name="front_axle_joint"
          type="revolute">
-    <origin xyz="0.4375 0 0"
+    <origin xyz="${base_x_origin_to_wheel_origin} 0 0"
             rpy="0 0 0" />
     <parent link="base_link" />
@@ -212,5 +212,5 @@
                  parent="front_axle_link"
                  translateX="0"
-                 translateY="1.75"
+                 translateY="1"
                  translateZ="0"
                  flipY="0" />
@@ -219,5 +219,5 @@
                  parent="front_axle_link"
                  translateX="0"
-                 translateY="-1.75"
+                 translateY="-1"
                  translateZ="0"
                  flipY="1" />

File: grizzly_description/urdf/wheel.urdf.xacro (robot description, xacro)
@@ -64,7 +64,7 @@
   <!-- at center of mass aligned with coordinate system, kg*m^2-->
   <property name="base_x_origin_to_wheel_origin"
-            value="0.25600006" />
+            value="0.448" />
   <property name="base_y_origin_to_wheel_origin"
-            value="0.285475" />
+            value="0.499" />
   <property name="base_z_origin_to_wheel_origin"
             value="0.0" />

Commit message: Remove add_frame.xacro. Add sensor links to the base.xacro

File: grizzly_description/urdf/base.urdf.xacro (robot description, xacro)
@@ -29,6 +29,4 @@
   <xacro:include filename="materials.urdf.xacro" />
   <xacro:include filename="wheel.urdf.xacro" />
-  <xacro:include filename="parts.urdf.xacro" />
-  <xacro:include filename="add_frame.urdf.xacro" />
   <xacro:include filename="grizzly.gazebo" />
   <!-- PROPERTY LIST -->
@@ -119,15 +117,25 @@
   </link>
   <!-- Add a sensor anchor link that points to the center of the robot top plate -->
-  <grizzly_tf parent="base_link" name="sensor_anchor_link"
-    translateX="0" translateY="0" translateZ="${chassis_height}"
-    rotateX="0" rotateY="0" rotateZ="0"/>
-  <!-- Add a sensor anchor link for the imu -->
-  <grizzly_tf parent="sensor_anchor_link" name="imu_link"
-    translateX="-${chassis_length/2}" translateY="0" translateZ="0"
-    rotateX="${M_PI}" rotateY="${M_PI/2}" rotateZ="0" />
-  <!-- Add a sensor anchor link for the gps -->
-  <grizzly_tf parent="sensor_anchor_link" name="navsat_link"
-    translateX="-${chassis_length/2}" translateY="0" translateZ="0"
-    rotateX="${M_PI}" rotateY="${M_PI/2}" rotateZ="0" />
+  <link name="sensor_anchor_link"/>
+  <joint name="sensor_anchor_joint" type="fixed">
+    <origin xyz="0 0 ${chassis_height}"
+            rpy="0 0 0" />
+    <parent link="base_link" />
+    <child link="sensor_anchor_link" />
+  </joint>
+  <link name="navsat_link" />
+  <joint name="navsat_joint" type="fixed">
+    <origin xyz="-${chassis_length/2} 0 0"
+            rpy="${M_PI} ${M_PI/2} 0" />
+    <parent link="sensor_anchor_link" />
+    <child link="navsat_link" />
+  </joint>
+  <link name="imu_link" />
+  <joint name="imu_joint" type="fixed">
+    <origin xyz="-${chassis_length/2} 0 0"
+            rpy="${M_PI} ${M_PI/2} 0" />
+    <parent link="sensor_anchor_link" />
+    <child link="imu_link" />
+  </joint>
   <!-- DECORATIONS -->
   <!-- Fenders -->

Commit message: Remove a bunch more indirection.
Mainly affects the inertia properties.

File: grizzly_description/urdf/base.urdf.xacro (robot description, xacro)
@@ -2,4 +2,5 @@
 <!--
 Copyright (c) 2012, Siddhant Ahuja (Sid), Ryan Gariepy
+Copyright (c) 2014, Clearpath Robotics
 All rights reserved.
 Redistribution and use in source and binary forms, with or without
@@ -26,55 +27,21 @@
 -->
 <robot name="grizzly" xmlns:xacro="http://www.ros.org/wiki/xacro">
+  <property name="M_PI" value="3.1415926535897931" />
+  <property name="ground_clearance" value="0.203" />
   <!-- Included URDF/XACRO Files -->
   <xacro:include filename="materials.urdf.xacro" />
   <xacro:include filename="wheel.urdf.xacro" />
   <xacro:include filename="grizzly.gazebo" />
-  <!-- PROPERTY LIST -->
-  <!--All units in m-kg-s-radians unit system -->
-  <property name="M_PI"
-            value="3.1415926535897931" />
-  <!-- Main Body-base-->
-  <!-- Location of com : center of mass -->
-  <property name="base_x_com"
-            value="-0.013" />
-  <property name="base_y_com"
-            value="-0.00061" />
-  <property name="base_z_com"
-            value="-0.0205" />
+  <!-- Key Dimensions -->
   <property name="chassis_length" value="1.75" />
   <property name="chassis_width" value="0.711" />
   <property name="chassis_height" value="0.495" />
-  <!-- Mass of the base-->
-  <property name="base_mass" value="487" />
-  <!-- Mass of the front axle-->
+  <property name="chassis_mass" value="487" />
   <property name="front_axle_mass" value="113" />
   <property name="front_axle_radius" value="0.13" />
   <property name="front_axle_length" value="1.0" />
-  <!-- Moments of inertia. Taken at center of mass aligned with coordinate system, kg*m^2-->
-  <!-- Ix = Iz = m*(3r^2 + h^2)/12   Iy = m*r^2/2-->
-  <property name="front_axle_ixx_com_cs"
-            value="9.9" />
-  <property name="front_axle_ixy_com_cs"
-            value="0.0" />
-  <property name="front_axle_ixz_com_cs"
-            value="0.0" />
-  <property name="front_axle_iyy_com_cs"
-            value="9.9" />
-  <property name="front_axle_iyz_com_cs"
-            value="0.0" />
-  <property name="front_axle_izz_com_cs"
-            value="0.95" />
-  <property name="base_ixx_com_cs"
-            value="64.010712692" />
-  <property name="base_ixy_com_cs"
-            value="0.214224647" />
-  <property name="base_ixz_com_cs"
-            value="-1.636784296" />
-  <property name="base_iyy_com_cs"
-            value="200.87" />
-  <property name="base_iyz_com_cs"
-            value="-0.048325439" />
-  <property name="base_izz_com_cs"
-            value="229.831441333" />
+  <property name="base_x_origin_to_wheel_origin" value="0.448" /> <!-- 240/2 + 660/2-->
+  <property name="base_y_origin_to_wheel_origin" value="0.499" /> <!--(1282-711)/4 + 711/2-->
+  <property name="base_z_origin_to_wheel_origin" value="0.0" />
   <!-- BASE-LINK -->
   <link name="base_link" />
@@ -90,13 +57,8 @@
   <link name="chassis_link">
     <inertial>
-      <mass value="${base_mass}" />
-      <!-- Center of mass -->
-      <origin xyz="${base_x_com} ${base_y_com} ${base_z_com}" />
-      <inertia ixx="${base_ixx_com_cs}"
-               ixy="${base_ixy_com_cs}"
-               ixz="${base_ixz_com_cs}"
-               iyy="${base_iyy_com_cs}"
-               iyz="${base_iyz_com_cs}"
-               izz="${base_izz_com_cs}" />
+      <mass value="${chassis_mass}"/>
+      <origin xyz="-0.013 -0.00061 -0.0205"/>
+      <inertia ixx="64.010712692" ixy="0.214224647" ixz="-1.636784296"
+               iyy="200.87" iyz="-0.048325439" izz="229.831441333" />
     </inertial>
     <visual>
@@ -154,18 +116,8 @@
   </joint>
   <!-- rear wheels -->
-  <grizzly_wheel fr="rear"
-                 lr="left"
-                 parent="chassis_link"
-                 translateX="-1"
-                 translateY="1"
-                 translateZ="0"
-                 flipY="0" />
-  <grizzly_wheel fr="rear"
-                 lr="right"
-                 parent="chassis_link"
-                 translateX="-1"
-                 translateY="-1"
-                 translateZ="0"
-                 flipY="1" />
+  <grizzly_wheel fr="rear" lr="left" flipY="0" parent="chassis_link"
+                 translateX="-1" translateY="1" />
+  <grizzly_wheel fr="rear" lr="right" flipY="1" parent="chassis_link"
+                 translateX="-1" translateY="-1" />
   <!-- Front axle link -->
   <joint name="front_axle_joint"
@@ -185,11 +137,6 @@
     <inertial>
       <mass value="${front_axle_mass}" />
-      <origin xyz="0 0 0" />
-      <inertia ixx="${front_axle_ixx_com_cs}"
-               ixy="${front_axle_ixy_com_cs}"
-               ixz="${front_axle_ixz_com_cs}"
-               iyy="${front_axle_iyy_com_cs}"
-               iyz="${front_axle_iyz_com_cs}"
-               izz="${front_axle_izz_com_cs}" />
+      <origin xyz="0 0 0"/>
+      <inertia ixx="9.9" ixy="0.0" ixz="0.0" iyy="9.9" iyz="0.0" izz="0.95" />
     </inertial>
     <visual>
@@ -211,17 +158,7 @@
   </link>
   <!-- Front wheels -->
-  <grizzly_wheel fr="front"
-                 lr="left"
-                 parent="front_axle_link"
-                 translateX="0"
-                 translateY="1"
-                 translateZ="0"
-                 flipY="0" />
-  <grizzly_wheel fr="front"
-                 lr="right"
-                 parent="front_axle_link"
-                 translateX="0"
-                 translateY="-1"
-                 translateZ="0"
-                 flipY="1" />
+  <grizzly_wheel fr="front" lr="left" parent="front_axle_link"
+                 translateX="0" translateY="1" flipY="0" />
+  <grizzly_wheel fr="front" lr="right" parent="front_axle_link"
+                 translateX="0" translateY="-1" flipY="1" />
 </robot>

File: grizzly_description/urdf/wheel.urdf.xacro (robot description, xacro)
@@ -2,4 +2,5 @@
 <!--
 Copyright (c) 2012, Siddhant Ahuja (Sid)
+Copyright (c) 2014, Clearpath Robotics
 All rights reserved.
 Redistribution and use in source and binary forms, with or without
@@ -26,53 +27,16 @@
 -->
 <robot name="grizzly_wheel" xmlns:xacro="http://ros.org/wiki/xacro">
-  <property name="M_PI"
-            value="3.14159" />
-  <!-- Wheel -->
   <property name="wheel_mass" value="15" />
-  <property name="wheel_radius"
-            value="0.33" />
-  <property name="wheel_width"
-            value="0.252" />
-  <!-- com : center of mass -->
-  <property name="wheel_x_com"
-            value="-0.002" />
-  <property name="wheel_y_com"
-            value="-0.198" />
-  <property name="wheel_z_com"
-            value="0.003" />
-  <!-- Moments of inertia. Taken at center of mass aligned with coordinate system, kg*m^2-->
-  <property name="wheel_ixx_com_cs"
-            value="14.68" />
-  <property name="wheel_ixy_com_cs"
-            value="-0.033" />
-  <property name="wheel_ixz_com_cs"
-            value="0.070" />
-  <property name="wheel_iyy_com_cs"
-            value="26.7" />
-  <property name="wheel_iyz_com_cs"
-            value="-0.05" />
-  <property name="wheel_izz_com_cs"
-            value="14.68" />
-  <property name="base_x_origin_to_wheel_origin"
-            value="0.448" /> <!-- 240/2 + 660/2-->
-  <property name="base_y_origin_to_wheel_origin"
-            value="0.499" /> <!--(1282-711)/4 + 711/2-->
-  <property name="base_z_origin_to_wheel_origin"
-            value="0.0" />
-  <property name="ground_clearance"
-            value="0.203" />
+  <property name="wheel_radius" value="0.33" />
+  <property name="wheel_width" value="0.252" />
   <xacro:macro name="grizzly_wheel"
-               params="fr lr parent translateX translateY translateZ flipY">
+               params="fr lr parent translateX translateY flipY">
     <!--fr : front, rear ; lr: left, right -->
     <link name="${fr}_${lr}_wheel">
       <inertial>
         <mass value="${wheel_mass}" />
-        <origin xyz="${wheel_x_com} ${wheel_y_com} ${wheel_z_com}" />
-        <inertia ixx="${wheel_ixx_com_cs}"
-                 ixy="${wheel_ixy_com_cs}"
-                 ixz="${wheel_ixz_com_cs}"
-                 iyy="${wheel_iyy_com_cs}"
-                 iyz="${wheel_iyz_com_cs}"
-                 izz="${wheel_izz_com_cs}" />
+        <origin xyz="-0.002 -0.198 0.003" />
+        <inertia ixx="14.68" ixy="-0.033" ixz="0.07"
+                 iyy="26.7" iyz="-0.05" izz="14.68" />
       </inertial>
       <visual>
@@ -107,5 +71,5 @@
       <parent link="${parent}" />
       <child link="${fr}_${lr}_wheel" />
-      <origin xyz="${translateX * base_x_origin_to_wheel_origin} ${translateY * base_y_origin_to_wheel_origin} ${translateZ}"
+      <origin xyz="${translateX * base_x_origin_to_wheel_origin} ${translateY * base_y_origin_to_wheel_origin} 0"
               rpy="0 0 0" />
       <axis xyz="0 1 0"
@@ -116,5 +80,5 @@
                         friction="0.0" />
     </joint>
-    <!-- Transmission is important to link the joints and the controller -->
+    <!-- Transmission links the joints and the controller -->
 <!--     <transmission name="joint_${fr}_${lr}_wheel_trans"
                   type="SimpleTransmission">

Commit message: small fix

File: grizzly_description/urdf/base.urdf.xacro (robot description, xacro)
@@ -81,6 +81,6 @@
   <joint name="base_link_joint"
          type="fixed">
-    <origin xyz="0 0 0"
-            rpy="0 0 ${ground_clearance}"/>
+    <origin xyz="0 0 ${ground_clearance}"
+            rpy="0 0 0"/>
     <parent link="base_link" />
     <child link="chassis_link" />
