Commit message: A few more tidy-ups here.
- More joints to after their respective child links.
- Group wheels together at the end.
- Re-add IMU orientation.

File: grizzly_description/urdf/base.urdf.xacro (robot description, xacro)
@@ -44,15 +44,7 @@
   <property name="base_y_origin_to_wheel_origin" value="0.499" /> <!--(1282-711)/4 + 711/2-->
   <property name="base_z_origin_to_wheel_origin" value="0.0" />
-  <!-- BASE-LINK -->
+  <!-- Root link of Grizzly -->
   <link name="base_link" />
-  <joint name="base_link_joint"
-         type="fixed">
-    <origin xyz="0 0 ${ground_clearance}"
-            rpy="0 0 0"/>
-    <parent link="base_link" />
-    <child link="chassis_link" />
-  </joint>
-  <!-- CHASSIS-LINK -->
-  <!--Actual body/chassis of the robot-->
+  <!-- Actual body/chassis of the robot, separate from base_link due to KDL inertia issue. -->
   <link name="chassis_link">
     <inertial>
@@ -74,8 +66,15 @@
               rpy="${M_PI/2} 0 ${M_PI/2}" />
       <geometry>
-         <box size="${chassis_width} ${chassis_height} ${chassis_length}"/>
+         <box size="${chassis_width} ${chassis_height} ${chassis_length}" />
       </geometry>
     </collision>
   </link>
+  <joint name="chassis_joint"
+         type="fixed">
+    <origin xyz="0 0 ${ground_clearance}"
+            rpy="0 0 0"/>
+    <parent link="base_link" />
+    <child link="chassis_link" />
+  </joint>
   <!-- Add a sensor anchor link that points to the center of the robot top plate -->
   <link name="sensor_anchor_link"/>
@@ -86,4 +85,5 @@
     <child link="sensor_anchor_link" />
   </joint>
+  <!-- This is the approximate position of the GPS antenna on the standard configuration. -->
   <link name="navsat_link" />
   <joint name="navsat_joint" type="fixed">
@@ -93,13 +93,13 @@
     <child link="navsat_link" />
   </joint>
+  <!-- The position and orientation of the IMU in the rear compartment. -->
   <link name="imu_link" />
   <joint name="imu_joint" type="fixed">
     <origin xyz="-${chassis_length/2} 0 0"
-            rpy="0 0 0" />
+            rpy="${M_PI} ${M_PI/2} 0" />
     <parent link="sensor_anchor_link" />
     <child link="imu_link" />
   </joint>
-  <!-- DECORATIONS -->
-  <!-- Fenders -->
+  <!-- Purely decorative visual component. -->
   <link name="fenders_link">
     <visual>
@@ -114,23 +114,4 @@
     <parent link="chassis_link" />
     <child link="fenders_link" />
-  </joint>
-  <!-- rear wheels -->
-  <grizzly_wheel fr="rear" lr="left" flipY="0" parent="chassis_link"
-                 translateX="-1" translateY="1" />
-  <grizzly_wheel fr="rear" lr="right" flipY="1" parent="chassis_link"
-                 translateX="-1" translateY="-1" />
-  <!-- Front axle link -->
-  <joint name="front_axle_joint"
-         type="revolute">
-    <origin xyz="${base_x_origin_to_wheel_origin} 0 0"
-            rpy="0 0 0" />
-    <parent link="chassis_link" />
-    <child link="front_axle_link" />
-    <axis xyz="1 0 0"
-          rpy="0 0 0" />
-    <limit effort="10"
-           lower="-0.2"
-           upper="0.2"
-           velocity="0.5" />
   </joint>
   <link name="front_axle_link">
@@ -157,8 +138,24 @@
     </collision>
   </link>
-  <!-- Front wheels -->
+  <joint name="front_axle_joint"
+         type="revolute">
+    <origin xyz="${base_x_origin_to_wheel_origin} 0 0"
+            rpy="0 0 0" />
+    <parent link="chassis_link" />
+    <child link="front_axle_link" />
+    <axis xyz="1 0 0"
+          rpy="0 0 0" />
+    <limit effort="10"
+           lower="-0.2"
+           upper="0.2"
+           velocity="0.5" />
+  </joint>
   <grizzly_wheel fr="front" lr="left" parent="front_axle_link"
                  translateX="0" translateY="1" flipY="0" />
   <grizzly_wheel fr="front" lr="right" parent="front_axle_link"
                  translateX="0" translateY="-1" flipY="1" />
+  <grizzly_wheel fr="rear" lr="left" parent="chassis_link"
+                 translateX="-1" translateY="1" flipY="0" />
+  <grizzly_wheel fr="rear" lr="right" parent="chassis_link"
+                 translateX="-1" translateY="-1" flipY="1" />
 </robot>

Commit message: Fix IMU origin.
IMU origin is set as it is mount on real robot. But in imu controller plugin in simulation the frameID is set to base_link.

File: grizzly_description/urdf/base.urdf.xacro (robot description, xacro)
@@ -121,5 +121,5 @@
     <origin xyz="0 0 ${chassis_height}"
             rpy="0 0 0" />
-    <parent link="base_link" />
+    <parent link="chassis_link" />
     <child link="sensor_anchor_link" />
   </joint>
@@ -133,6 +133,6 @@
   <link name="imu_link" />
   <joint name="imu_joint" type="fixed">
-    <origin xyz="-${chassis_length/2} 0 0"
-            rpy="0 0 0" />
+    <origin xyz="-${chassis_length/2} 0 -${chassis_height/2}"
+             rpy="${M_PI} ${M_PI/2} 0" />
     <parent link="sensor_anchor_link" />
     <child link="imu_link" />

Commit message: Update to match Cuddles configurations.

File: grizzly_description/urdf/base.urdf.xacro (robot description, xacro)
@@ -104,5 +104,5 @@
   <xacro:if value="$(arg spawn_lidar)">
     <xacro:include filename="$(find grizzly_description)/urdf/lidar.urdf.xacro"/>
-    <xacro:lidar_sensor name="lidar" parent="sensor_anchor_link" ros_topic="lidar_scan"
+    <xacro:lidar_sensor name="lidar" parent="sensor_anchor_link" ros_topic="scan"
       update_rate="20" x="0" y="0" z="${chassis_height/2-0.2}" r="0" p="0" yaw="0" samples="500"
       min_angle="-1.57" max_angle="1.57" min_range="0.3" max_range="20" resolution="0.05"

File: grizzly_description/urdf/lidar.gazebo.xacro (robot description, xacro)
@@ -2,5 +2,5 @@
 <robot xmlns:xacro="http://ros.org/wiki/xacro">
   <xacro:macro name="lidar_sensor_gazebo" params="name ros_topic update_rate samples min_angle max_angle min_range max_range resolution visible">
-    <gazebo reference="${name}_link">
+    <gazebo reference="laser">
       <sensor type="ray" name="${name}">
         <always_on>true</always_on>
@@ -28,5 +28,5 @@
           <updateRate>${update_rate}</updateRate>
           <topicName>${ros_topic}</topicName>
-          <frameName>${name}_link</frameName>
+          <frameName>laser</frameName>
         </plugin>
       </sensor>

File: grizzly_description/urdf/lidar.urdf.xacro (robot description, xacro)
@@ -3,5 +3,5 @@
   <xacro:include filename="$(find grizzly_description)/urdf/lidar.gazebo.xacro"/>
   <xacro:macro name="lidar_sensor" params="name parent ros_topic update_rate x y z r p yaw samples min_angle max_angle min_range max_range resolution visible">
-  <link name="${name}_link">
+    <link name="laser">
     <inertial>
       <mass value = "0.2" />
@@ -19,7 +19,7 @@
     <origin xyz="${x} ${y} ${z}" rpy="${r} ${p} ${yaw}"/>
     <parent link="${parent}"/>
-    <child link="${name}_link"/>
+    <child link="laser"/>
   </joint>
-  <gazebo reference="${name}_link">
+  <gazebo reference="laser">
     <material>Gazebo/Blue</material>
   </gazebo>
