Commit message: Fix vehicle dimensions for roscontrol

File: grizzly_description/urdf/grizzly.urdf.xacro (robot description, xacro)
@@ -17,10 +17,10 @@
   <xacro:property name="front_axle_length" value="1.0" />
   <xacro:property name="wheelbase" value="0.896" />
-  <xacro:property name="track" value="0.499" />
+  <xacro:property name="track" value="0.537" />
   <!-- Wheel Mounting Positions -->
   <xacro:property name="wheel_vertical_offset" value="0.03282" />
   <!-- Wheel Properties -->
-  <xacro:property name="wheel_width" value="0.252" />
-  <xacro:property name="wheel_radius" value="0.33" />
+  <xacro:property name="wheel_width" value="0.2667" />
+  <xacro:property name="wheel_radius" value="0.3175" />
   <xacro:property name="wheel_mass" value="15" />
   <!-- Root link of Grizzly -->
@@ -55,6 +55,6 @@
     </inertial>
     <visual>
-      <origin xyz="-${ground_clearance} 0.01 ${track}"
-              rpy="0 ${M_PI} ${M_PI/2}" />
+      <origin xyz="0 0 0"
+              rpy="0 0 0" />
       <geometry>
         <mesh filename="package://grizzly_description/meshes/front_axle.stl" />
@@ -153,14 +153,14 @@
   <!-- Grizzly wheel macros -->
   <xacro:grizzly_wheel wheel_prefix="front_left" parent="front_axle_link" flipY="0">
-    <origin xyz="0 0.499 ${wheel_vertical_offset}" rpy="0 0 0" />
+    <origin xyz="0 ${track} ${wheel_vertical_offset}" rpy="0 0 0" />
   </xacro:grizzly_wheel>
   <xacro:grizzly_wheel wheel_prefix="front_right" parent="front_axle_link" flipY="1">
-    <origin xyz="0 -0.499 ${wheel_vertical_offset}" rpy="0 0 0" />
+    <origin xyz="0 ${-track} ${wheel_vertical_offset}" rpy="0 0 0" />
   </xacro:grizzly_wheel>
   <xacro:grizzly_wheel wheel_prefix="rear_left" parent="chassis_link" flipY="0">
-    <origin xyz="-0.448 0.499 ${wheel_vertical_offset}" rpy="0 0 0" />
+    <origin xyz="${-wheelbase/2} ${track} ${wheel_vertical_offset}" rpy="0 0 0" />
   </xacro:grizzly_wheel>
   <xacro:grizzly_wheel wheel_prefix="rear_right" parent="chassis_link" flipY="1">
-    <origin xyz="-0.448 -0.499 ${wheel_vertical_offset}" rpy="0 0 0" />
+    <origin xyz="${-wheelbase/2} ${-track} ${wheel_vertical_offset}" rpy="0 0 0" />
   </xacro:grizzly_wheel>
   <xacro:grizzly_decorate />

Commit message: Updated urdf to have both sensor arches, all standard sensors, and some non-standard sensors

File: grizzly_description/urdf/grizzly.urdf.xacro (robot description, xacro)
@@ -26,4 +26,11 @@
   <!-- Root link of Grizzly -->
   <link name="base_link" />
+  <!-- Sensor Arch Options -->
+  <xacro:arg name="front_sensor_arch_enabled" default="$(optenv GRIZZLY_FRONT_SENSOR_ARCH_ENABLED false)" />
+  <xacro:arg name="front_tower_xyz" default="$(optenv GRIZZLY_FRONT_SENSOR_ARCH_XYZ 0.495 0.0 0.0)" />
+  <xacro:arg name="front_tower_rpy" default="$(optenv GRIZZLY_FRONT_SENSOR_ARCH_RPY 0.0 0.0 0.0)" />
+  <xacro:arg name="rear_sensor_arch_enabled" default="$(optenv GRIZZLY_REAR_SENSOR_ARCH_ENABLED true)" />
+  <xacro:arg name="rear_tower_xyz" default="$(optenv GRIZZLY_REAR_SENSOR_ARCH_XYZ -0.63 0.0 0.0)" />
+  <xacro:arg name="rear_tower_rpy" default="$(optenv GRIZZLY_REAR_SENSOR_ARCH_RPY 0.0 0.0 0.0)" />
   <!-- Base link is the center of the robot's bottom plate -->
   <link name="chassis_link">
@@ -98,12 +105,4 @@
     <child link="sensor_anchor_link" />
   </joint>
-  <!-- This is the approximate position of the GPS antenna on the standard configuration. -->
-  <link name="navsat_link" />
-  <joint name="navsat_joint" type="fixed">
-    <origin xyz="-${base_x_size/2} 0 0"
-            rpy="0 0 0" />
-    <parent link="sensor_anchor_link" />
-    <child link="navsat_link" />
-  </joint>
   <!-- The position and orientation of the IMU in the rear compartment. -->
   <link name="imu_link" />
@@ -126,4 +125,5 @@
 			    <mesh filename="package://grizzly_description/meshes/wheel.stl" />
 			  </geometry>
+        <material name="DarkGrey" />
 			</visual>
 			<collision>
@@ -164,4 +164,126 @@
     <origin xyz="${-wheelbase/2} ${-track} ${wheel_vertical_offset}" rpy="0 0 0" />
   </xacro:grizzly_wheel>
+  <!-- Front Sensor Arch -->
+  <xacro:if value="$(arg front_sensor_arch_enabled)">
+    <link name="front_sensor_base_link">
+      <visual>
+        <origin xyz="0 0 0" rpy="0 0 0" />
+        <geometry>
+          <mesh filename="package://grizzly_description/meshes/sensor_risers.stl" />
+        </geometry>
+        <material name="DarkGrey" />
+      </visual>
+      <collision>
+        <geometry>
+          <mesh filename="package://grizzly_description/meshes/sensor_risers.stl" />
+        </geometry>
+      </collision>
+    </link>
+    <joint name="front_sensor_base_joint" type="fixed">
+      <origin xyz="$(arg front_tower_xyz)" rpy="$(arg rear_tower_rpy)" />
+      <parent link="sensor_anchor_link" />
+      <child link="front_sensor_base_link" />
+    </joint>
+    <link name="front_sensor_arch_link">
+      <visual>
+        <origin xyz="0 0 0" rpy="0 0 0" />
+        <geometry>
+          <mesh filename="package://grizzly_description/meshes/sensor_arch.stl" />
+        </geometry>
+        <material name="DarkGrey" />
+      </visual>
+      <collision>
+        <geometry>
+          <mesh filename="package://grizzly_description/meshes/sensor_arch.stl" />
+        </geometry>
+      </collision>
+    </link>
+    <joint name="front_sensor_arch_joint" type="fixed">
+      <origin xyz="0 0 0.3" rpy="0 0 0" />
+      <parent link="front_sensor_base_link" />
+      <child link="front_sensor_arch_link" />
+    </joint>
+    <link name="front_sensor_mount_link"/>
+    <joint name="front_sensor_mount_joint" type="fixed">
+      <origin xyz="0 0 0.15" rpy="0 0 0" />
+      <parent link="front_sensor_arch_link" />
+      <child link="front_sensor_mount_link" />
+    </joint>
+  </xacro:if>
+  <link name="navsat_link" />
+  <!-- Rear Sensor Arch -->
+  <xacro:if value="$(arg rear_sensor_arch_enabled)">
+    <link name="rear_sensor_base_link">
+      <visual>
+        <origin xyz="0 0 0" rpy="0 0 0" />
+        <geometry>
+          <mesh filename="package://grizzly_description/meshes/sensor_risers.stl" />
+        </geometry>
+        <material name="DarkGrey" />
+      </visual>
+      <collision>
+        <geometry>
+          <mesh filename="package://grizzly_description/meshes/sensor_risers.stl" />
+        </geometry>
+      </collision>
+    </link>
+    <joint name="rear_sensor_base_joint" type="fixed">
+      <origin xyz="$(arg rear_tower_xyz)" rpy="$(arg rear_tower_rpy)" />
+      <parent link="sensor_anchor_link" />
+      <child link="rear_sensor_base_link" />
+    </joint>
+    <link name="rear_sensor_plate_link">
+      <visual>
+        <origin xyz="0 0 0" rpy="0 0 0" />
+        <geometry>
+          <mesh filename="package://grizzly_description/meshes/sensor_plate.stl" />
+        </geometry>
+        <material name="DarkGrey" />
+      </visual>
+      <collision>
+        <geometry>
+          <mesh filename="package://grizzly_description/meshes/sensor_plate.stl" />
+        </geometry>
+      </collision>
+    </link>
+    <joint name="rear_sensor_plate_joint" type="fixed">
+      <origin xyz="0 0 0.3" rpy="0 0 0" />
+      <parent link="rear_sensor_base_link" />
+      <child link="rear_sensor_plate_link" />
+    </joint>
+    <link name="rear_antenna_link">
+      <visual>
+        <origin xyz="0 0 0" rpy="0 0 0" />
+        <geometry>
+          <mesh filename="package://grizzly_description/meshes/antennas.stl" />
+        </geometry>
+        <material name="Grey" />
+      </visual>
+      <collision>
+        <geometry>
+          <mesh filename="package://grizzly_description/meshes/antennas.stl" />
+        </geometry>
+      </collision>
+    </link>
+    <joint name="rear_antenna_joint" type="fixed">
+      <origin xyz="0 0 0.003175" rpy="0 0 0" />
+      <parent link="rear_sensor_plate_link" />
+      <child link="rear_antenna_link" />
+    </joint>
+    <!-- This is the approximate position of the GPS antenna on the standard configuration. -->
+    <joint name="navsat_joint" type="fixed">
+      <origin xyz="0 0 0.4" rpy="0 0 0" />
+      <parent link="rear_sensor_plate_link" />
+      <child link="navsat_link" />
+    </joint>
+  </xacro:if>
+  <xacro:unless value="$(arg rear_sensor_arch_enabled)">
+    <joint name="navsat_joint" type="fixed">
+      <origin xyz="-${base_x_size/2} 0 0"
+              rpy="0 0 0" />
+      <parent link="sensor_anchor_link" />
+      <child link="navsat_link" />
+    </joint>
+  </xacro:unless>
   <xacro:grizzly_decorate />
   <!-- Bring in simulation data for Gazebo. -->

Commit message: URDF formatting

File: grizzly_description/urdf/grizzly.urdf.xacro (robot description, xacro)
@@ -113,42 +113,42 @@
     <child link="imu_link" />
   </joint>
-	<xacro:macro name="grizzly_wheel" params="wheel_prefix parent *joint_pose flipY">
-		<link name="${wheel_prefix}_wheel_link">
-			<inertial>
-			  <mass value="${wheel_mass}" />
-			  <origin xyz="-0.002 -0.198 0.003" />
-			  <inertia  ixx="14.68" ixy="-0.033" ixz="0.07" iyy="26.7" iyz="-0.05" izz="14.68" />
-			</inertial>
-			<visual>
-			  <origin xyz="0 0 0" rpy="${M_PI/2} ${flipY*M_PI} ${M_PI/2}" />
-			  <geometry>
-			    <mesh filename="package://grizzly_description/meshes/wheel.stl" />
-			  </geometry>
-        <material name="DarkGrey" />
-			</visual>
-			<collision>
-			  <origin xyz="0 0 0" rpy="${M_PI/2} ${flipY*M_PI} 0" />
-			  <geometry>
-		  	    <cylinder length="${wheel_width}" radius="${wheel_radius}" />
-			  </geometry>
-			</collision>
-		</link>
-		<joint name="${wheel_prefix}_wheel" type="continuous">
-			<parent link="${parent}"/>
-			<child link="${wheel_prefix}_wheel_link"/>
-			<xacro:insert_block name="joint_pose"/>
-			<axis xyz="0 1 0" rpy="0 0 0" />
-			<joint_properties damping="0.0" friction="0.0" />
-		</joint>
-		<transmission name="${wheel_prefix}_wheel_trans" type="SimpleTransmission">
-			<type>transmission_interface/SimpleTransmission</type>
-			<actuator name="${wheel_prefix}_wheel_motor">
-				<mechanicalReduction>1</mechanicalReduction>
-			</actuator>
-			<joint name="${wheel_prefix}_wheel">
-				<hardwareInterface>hardware_interface/VelocityJointInterface</hardwareInterface>
-			</joint>
-		</transmission>
-	</xacro:macro>
+  <xacro:macro name="grizzly_wheel" params="wheel_prefix parent *joint_pose flipY">
+    <link name="${wheel_prefix}_wheel_link">
+      <inertial>
+        <mass value="${wheel_mass}" />
+        <origin xyz="-0.002 -0.198 0.003" />
+        <inertia  ixx="14.68" ixy="-0.033" ixz="0.07" iyy="26.7" iyz="-0.05" izz="14.68" />
+      </inertial>
+      <visual>
+        <origin xyz="0 0 0" rpy="${M_PI/2} ${flipY*M_PI} ${M_PI/2}" />
+        <geometry>
+          <mesh filename="package://grizzly_description/meshes/wheel.stl" />
+        </geometry>
+        <material name="DarkGrey" />
+      </visual>
+      <collision>
+        <origin xyz="0 0 0" rpy="${M_PI/2} ${flipY*M_PI} 0" />
+        <geometry>
+          <cylinder length="${wheel_width}" radius="${wheel_radius}" />
+        </geometry>
+      </collision>
+    </link>
+    <joint name="${wheel_prefix}_wheel" type="continuous">
+      <parent link="${parent}"/>
+      <child link="${wheel_prefix}_wheel_link"/>
+      <xacro:insert_block name="joint_pose"/>
+      <axis xyz="0 1 0" rpy="0 0 0" />
+      <joint_properties damping="0.0" friction="0.0" />
+    </joint>
+    <transmission name="${wheel_prefix}_wheel_trans" type="SimpleTransmission">
+      <type>transmission_interface/SimpleTransmission</type>
+      <actuator name="${wheel_prefix}_wheel_motor">
+        <mechanicalReduction>1</mechanicalReduction>
+      </actuator>
+      <joint name="${wheel_prefix}_wheel">
+        <hardwareInterface>hardware_interface/VelocityJointInterface</hardwareInterface>
+      </joint>
+    </transmission>
+  </xacro:macro>
   <!-- Grizzly wheel macros -->
   <xacro:grizzly_wheel wheel_prefix="front_left" parent="front_axle_link" flipY="0">
